Commit message: claude tool updates

File: generated/IRB1520ID_4_150_v1/IRB1520ID_4_150.urdf (robot description, URDF)
Before this commit: robot CRB15000_12_127, 7 links, 6 joints
Links:
- link base_link: mass 43.32183458222497 -> 173.23686098491044
- link link_1_1: mass 41.02561837016391 -> 140.431105262512
- link link_2_1: mass 70.93334568132663 -> 41.09408994963129
- link link_3_1: mass 26.38179204175825 -> 87.68237861319876
- link link_4_1: mass 27.702603279655857 -> 21.10958519516661
- link link_5_1: mass 23.637515690396576 -> 4.145062543835652
- link link_6_1: mass 1.1500357263477234 -> 0.7222246780605773
Joints:
- joint j1: axis 0.0 -0.0 1.0 -> -0.0 -0.0 1.0; origin xyz=0.651068 0.882174 1.382204 rpy=0 0 0 -> xyz=0.0 0.0 0.179 rpy=0 0 0
- joint j2: axis 0.0 -1.0 0.0 -> 0.0 -1.0 -0.0; origin xyz=-0.00025 -0.09515 0.1231 rpy=0 0 0 -> xyz=0.16 -0.101 0.274 rpy=0 0 0
- joint j3: axis -0.0 1.0 -0.0 -> 0.0 -1.0 -0.0; origin xyz=0.0 0.00985 0.706969 rpy=0 0 0 -> xyz=0.0 -0.02 0.59 rpy=0 0 0
- joint j4: axis 1.0 -0.0 0.0 -> -1.0 -0.0 0.0; origin xyz=0.096 0.085 0.11 rpy=0 0 0 -> xyz=0.217 0.121676 0.2 rpy=0 0 0
- joint j5: axis 0.0 -1.0 0.0 -> 0.0 -1.0 -0.0; origin xyz=0.436883 0.0755 0.0 rpy=0 0 0 -> xyz=0.506 0.051824 0.0 rpy=0 0 0
- joint j6: axis 1.0 -0.0 0.0 -> 1.0 0.0 0.0; origin xyz=0.068 -0.0745 0.08 rpy=0 0 0 -> xyz=0.189629 -0.0525 0.0 rpy=0 0 0
