Commit message: Validation, limits, and robot improvements
- Add joint limits to all robot models
- Standardize mesh naming conventions (link_1, link_2, etc.)
- Fix joint limits and axis orientations
- Add URDF validation tool
- Update README with robot table and validation info
- Add IK demo scripts and utilities
- Improve documentation and project structure

🤖 Generated with [Claude Code](https://claude.ai/code)

Co-Authored-By: Claude <noreply@anthropic.com>

File: generated/CRB15000_10kg_152_v1/CRB15000_10kg_152.urdf (robot description, URDF)
Before this commit: robot CRB15000_10kg_152, 7 links, 6 joints
Links:
- removed link link_1_1
- removed link link_2_1
- removed link link_3_1
- removed link link_4_1
- removed link link_5_1
- removed link link_6_1
- added link flange, mass 0.1
- added link link_1, mass 62.519803241843114; collision mesh filename=meshes/link_1_1.stl scale=0.001 0.001 0.001; visual mesh filename=meshes/link_1_1.stl scale=0.001 0.001 0.001
- added link link_2, mass 70.93354798589783; collision mesh filename=meshes/link_2_1.stl scale=0.001 0.001 0.001; visual mesh filename=meshes/link_2_1.stl scale=0.001 0.001 0.001
- added link link_3, mass 26.381731962599385; collision mesh filename=meshes/link_3_1.stl scale=0.001 0.001 0.001; visual mesh filename=meshes/link_3_1.stl scale=0.001 0.001 0.001
- added link link_4, mass 32.073735291819936; collision mesh filename=meshes/link_4_1.stl scale=0.001 0.001 0.001; visual mesh filename=meshes/link_4_1.stl scale=0.001 0.001 0.001
- added link link_5, mass 23.637549891653943; collision mesh filename=meshes/link_5_1.stl scale=0.001 0.001 0.001; visual mesh filename=meshes/link_5_1.stl scale=0.001 0.001 0.001
- added link link_6, mass 1.1500367477208804; collision mesh filename=meshes/link_6_1.stl scale=0.001 0.001 0.001; visual mesh filename=meshes/link_6_1.stl scale=0.001 0.001 0.001
- added link tool0, mass 0.01
Joints:
- removed joint j1
- removed joint j2
- removed joint j3
- removed joint j4
- removed joint j5
- removed joint j6
- added joint joint_1: type revolute, parent base_link, child link_1, origin xyz=0.0 0.0 0.215 rpy=0 0 0, axis 0.0 0.0 -1.0, limit lower=-4.712 upper=4.712 effort=450 velocity=2.094
- added joint joint_2: type revolute, parent link_1, child link_2, origin xyz=0.15 -0.09615 0.185014 rpy=0 0 0, axis 0.0 1.0 0.0, limit lower=-3.14159 upper=3.14159 effort=400 velocity=2.094
- added joint joint_3: type revolute, parent link_2, child link_3, origin xyz=0.0 0.01115 0.706986 rpy=0 0 0, axis 0.0 -1.0 0.0, limit lower=-1.483 upper=3.927 effort=160 velocity=2.181
- added joint joint_4: type revolute, parent link_3, child link_4, origin xyz=0.096 0.085 0.11 rpy=0 0 0, axis 1.0 0.0 0.0, limit lower=-3.14159 upper=3.14159 effort=60 velocity=3.491
- added joint joint_5: type revolute, parent link_4, child link_5, origin xyz=0.540883 0.0755 0.0 rpy=0 0 0, axis 0.0 -1.0 0.0, limit lower=-3.14159 upper=3.14159 effort=60 velocity=3.491
- added joint joint_6: type revolute, parent link_5, child link_6, origin xyz=0.068117 -0.0755 0.08 rpy=0 0 0, axis 1.0 0.0 0.0, limit lower=-4.712 upper=4.712 effort=60 velocity=3.491
- added joint joint_flange: type fixed, parent link_6, child flange, origin xyz=0 0 0 rpy=0 1.57 0
- added joint joint_tool0: type fixed, parent flange, child tool0, origin xyz=0 0 0 rpy=0 0 0

File: generated/CRB15000_12kg_127_v1/CRB15000_12kg_127.urdf (robot description, URDF)
Before this commit: robot CRB15000_12_127, 7 links, 6 joints
Links:
- removed link CRB15000_12kg_127_Omnicore_rev00_LINK01_CAD_1
- removed link CRB15000_12kg_127_Omnicore_rev00_LINK02_CAD_1
- removed link CRB15000_12kg_127_Omnicore_rev00_LINK03_CAD_1
- removed link CRB15000_12kg_127_Omnicore_rev00_LINK04_CAD_1
- removed link CRB15000_12kg_127_Omnicore_rev00_LINK05_CAD_1
- removed link CRB15000_12kg_127_Omnicore_rev00_LINK06_CAD_1
- added link flange, mass 0.1
- added link link_1, mass 41.02562588128756; collision mesh filename=meshes/CRB15000_12kg_127_Omnicore_rev00_LINK01_CAD_1.stl scale=0.001 0.001 0.001; visual mesh filename=meshes/CRB15000_12kg_127_Omnicore_rev00_LINK01_CAD_1.stl scale=0.001 0.001 0.001
- added link link_2, mass 70.93334832681374; collision mesh filename=meshes/CRB15000_12kg_127_Omnicore_rev00_LINK02_CAD_1.stl scale=0.001 0.001 0.001; visual mesh filename=meshes/CRB15000_12kg_127_Omnicore_rev00_LINK02_CAD_1.stl scale=0.001 0.001 0.001
- added link link_3, mass 26.381731962312585; collision mesh filename=meshes/CRB15000_12kg_127_Omnicore_rev00_LINK03_CAD_1.stl scale=0.001 0.001 0.001; visual mesh filename=meshes/CRB15000_12kg_127_Omnicore_rev00_LINK03_CAD_1.stl scale=0.001 0.001 0.001
- added link link_4, mass 27.702812566356673; collision mesh filename=meshes/CRB15000_12kg_127_Omnicore_rev00_LINK04_CAD_1.stl scale=0.001 0.001 0.001; visual mesh filename=meshes/CRB15000_12kg_127_Omnicore_rev00_LINK04_CAD_1.stl scale=0.001 0.001 0.001
- added link link_5, mass 23.63754989165508; collision mesh filename=meshes/CRB15000_12kg_127_Omnicore_rev00_LINK05_CAD_1.stl scale=0.001 0.001 0.001; visual mesh filename=meshes/CRB15000_12kg_127_Omnicore_rev00_LINK05_CAD_1.stl scale=0.001 0.001 0.001
- added link link_6, mass 1.1500367505463056; collision mesh filename=meshes/CRB15000_12kg_127_Omnicore_rev00_LINK06_CAD_1.stl scale=0.001 0.001 0.001; visual mesh filename=meshes/CRB15000_12kg_127_Omnicore_rev00_LINK06_CAD_1.stl scale=0.001 0.001 0.001
- added link tool0, mass 0.01
Joints:
- removed joint j1
- removed joint j2
- removed joint j3
- removed joint j4
- removed joint j5
- removed joint j6
- added joint joint_1: type revolute, parent base_link, child link_1, origin xyz=0.0 0.0 0.181677 rpy=0 0 0, axis -0.0 0.0 1.0, limit lower=-4.712 upper=4.712 effort=390 velocity=2.094
- added joint joint_2: type revolute, parent link_1, child link_2, origin xyz=0.0 -0.09615 0.156323 rpy=0 0 0, axis 0.0 -1.0 -0.0, limit lower=-3.14159 upper=3.14159 effort=400 velocity=2.094
- added joint joint_3: type revolute, parent link_2, child link_3, origin xyz=0.0 0.00985 0.707 rpy=0 0 0, axis 0.0 -1.0 -0.0, limit lower=-3.927 upper=1.483 effort=160 velocity=2.181
- added joint joint_4: type revolute, parent link_3, child link_4, origin xyz=0.097 0.0863 0.11 rpy=0 0 0, axis -1.0 0.0 -0.0, limit lower=-3.14159 upper=3.14159 effort=60 velocity=3.491
- added joint joint_5: type revolute, parent link_4, child link_5, origin xyz=0.437 0.0745 0.0 rpy=0 0 0, axis 0.0 -1.0 0.0, limit lower=-3.14159 upper=3.14159 effort=60 velocity=3.491
- added joint joint_6: type revolute, parent link_5, child link_6, origin xyz=0.0685 -0.0745 0.08 rpy=0 0 0, axis -1.0 0.0 -0.0, limit lower=-4.712 upper=4.712 effort=60 velocity=3.491
- added joint joint_flange: type fixed, parent link_6, child flange, origin xyz=0 0 0 rpy=0 1.57 0
- added joint joint_tool0: type fixed, parent flange, child tool0, origin xyz=0 0 0 rpy=0 0 0

File: generated/CRB15000_5kg_950_v1/CRB15000_5kg_950.urdf (robot description, URDF)
Before this commit: robot CRB15000_5kg_950, 7 links, 6 joints
Links:
- removed link link_1_1
- removed link link_2_1
- removed link link_3_1
- removed link link_4_1
- removed link link_5_1
- removed link link_6_1
- added link flange, mass 0.1
- added link link_1, mass 21.72390566115484; collision mesh filename=meshes/link_1.stl scale=0.001 0.001 0.001; visual mesh filename=meshes/link_1.stl scale=0.001 0.001 0.001
- added link link_2, mass 33.66814621553652; collision mesh filename=meshes/link_2.stl scale=0.001 0.001 0.001; visual mesh filename=meshes/link_2.stl scale=0.001 0.001 0.001
- added link link_3, mass 26.559534737331685; collision mesh filename=meshes/link_3.stl scale=0.001 0.001 0.001; visual mesh filename=meshes/link_3.stl scale=0.001 0.001 0.001
- added link link_4, mass 21.811589078670252; collision mesh filename=meshes/link_4.stl scale=0.001 0.001 0.001; visual mesh filename=meshes/link_4.stl scale=0.001 0.001 0.001
- added link link_5, mass 23.63690573076678; collision mesh filename=meshes/link_5.stl scale=0.001 0.001 0.001; visual mesh filename=meshes/link_5.stl scale=0.001 0.001 0.001
- added link link_6, mass 1.1500367477202385; collision mesh filename=meshes/link_6.stl scale=0.001 0.001 0.001; visual mesh filename=meshes/link_6.stl scale=0.001 0.001 0.001
- added link tool0, mass 0.01
Joints:
- removed joint j1
- removed joint j2
- removed joint j3
- removed joint j4
- removed joint j5
- removed joint j6
- added joint joint_1: type revolute, parent base_link, child link_1, origin xyz=0.0 0.0 0.1885 rpy=0 0 0, axis 0.0 0.0 -1.0, limit lower=3.14159 upper=-3.14159 effort=175.44 velocity=2.181
- added joint joint_2: type revolute, parent link_1, child link_2, origin xyz=-0.0 -0.085 0.0765 rpy=0 0 0, axis 0.0 -1.0 0.0, limit lower=3.14159 upper=-3.14159 effort=175.44 velocity=2.181
- added joint joint_3: type revolute, parent link_2, child link_3, origin xyz=0.0 -0.001 0.444 rpy=0 0 0, axis 0.0 -1.0 0.0, limit lower=-3.927 upper=1.483 effort=90.6 velocity=2.444
- added joint joint_4: type revolute, parent link_3, child link_4, origin xyz=0.096 0.086 0.11 rpy=0 0 0, axis 1.0 0.0 0.0, limit lower=3.14159 upper=-3.14159 effort=18.72 velocity=3.491
- added joint joint_5: type revolute, parent link_4, child link_5, origin xyz=0.374 0.0745 0.0 rpy=0 0 0, axis 0.0 -1.0 0.0, limit lower=3.14159 upper=-3.14159 effort=21.44 velocity=3.491
- added joint joint_6: type revolute, parent link_5, child link_6, origin xyz=0.068 -0.0745 0.08 rpy=0 0 0, axis 1.0 0.0 0.0, limit lower=-4.712 upper=4.712 effort=9.2 velocity=3.491
- added joint joint_flange: type fixed, parent link_6, child flange, origin xyz=0 0 0 rpy=0 1.57 0
- added joint joint_tool0: type fixed, parent flange, child tool0, origin xyz=0 0 0 rpy=0 0 0

File: generated/IRB1100_4kg_475_STD_v1/IRB1100_4kg_475_STD.urdf (robot description, URDF)
Before this commit: robot IRB1100_4kg_475_STD, 7 links, 6 joints
Links:
- removed link link_1_1
- removed link link_2_1
- removed link link_3_1
- removed link link_4_1
- removed link link_5_1
- removed link link_6_1
- added link flange
- added link link_1, mass 24.887771906712818; collision mesh filename=meshes/link_1.stl scale=0.001 0.001 0.001; visual mesh filename=meshes/link_1.stl scale=0.001 0.001 0.001
- added link link_2, mass 17.325080500260935; collision mesh filename=meshes/link_2.stl scale=0.001 0.001 0.001; visual mesh filename=meshes/link_2.stl scale=0.001 0.001 0.001
- added link link_3, mass 8.02511707118897; collision mesh filename=meshes/link_3.stl scale=0.001 0.001 0.001; visual mesh filename=meshes/link_3.stl scale=0.001 0.001 0.001
- added link link_4, mass 10.264284403829079; collision mesh filename=meshes/link_4.stl scale=0.001 0.001 0.001; visual mesh filename=meshes/link_4.stl scale=0.001 0.001 0.001
- added link link_5, mass 2.582057596654616; collision mesh filename=meshes/link_5.stl scale=0.001 0.001 0.001; visual mesh filename=meshes/link_5.stl scale=0.001 0.001 0.001
- added link link_6, mass 0.05751158667684128; collision mesh filename=meshes/link_6.stl scale=0.001 0.001 0.001; visual mesh filename=meshes/link_6.stl scale=0.001 0.001 0.001
- added link tool0
Joints:
- removed joint j1
- removed joint j2
- removed joint j3
- removed joint j4
- removed joint j5
- removed joint j6
- added joint flange-tool0: type fixed, parent flange, child tool0, origin xyz=0.0 0.0 0.0 rpy=0 0 0
- added joint joint_1: type revolute, parent base_link, child link_1, origin xyz=0.0 0.0 0.146 rpy=0 0 0, axis 0.0 0.0 1.0, limit lower=-4.014 upper=4.014 effort=0.0 velocity=8.03
- added joint joint_2: type revolute, parent link_1, child link_2, origin xyz=0.0 -0.0525 0.181 rpy=0 0 0, axis 0.0 -1.0 0.0, limit lower=-2.007 upper=1.972 effort=0.0 velocity=6.28
- added joint joint_3: type revolute, parent link_2, child link_3, origin xyz=0.0 -0.0105 0.225 rpy=0 0 0, axis 0.0 -1.0 0.0, limit lower=-3.577 upper=0.960 effort=0.0 velocity=4.89
- added joint joint_4: type revolute, parent link_3, child link_4, origin xyz=0.0725 0.063 0.01 rpy=0 0 0, axis 1.0 0.0 0.0, limit lower=-4.014 upper=4.014 effort=0.0 velocity=9.77
- added joint joint_5: type revolute, parent link_4, child link_5, origin xyz=0.1775 0.0265 0.0 rpy=0 0 0, axis 0.0 -1.0 0.0, limit lower=-2.181 upper=2.094 effort=0.0 velocity=7.33
- added joint joint_6: type revolute, parent link_5, child link_6, origin xyz=0.056 -0.0265 0.0 rpy=0 0 0, axis -1.0 0.0 0.0, limit lower=-6.981 upper=6.981 effort=0.0 velocity=13.09
- added joint joint_6-flange: type fixed, parent link_6, child flange, origin xyz=0.0 0.0 0.0 rpy=0 1.57 0

File: generated/IRB1100_4kg_580_STD_v1/IRB1100_4kg_580_STD.urdf (robot description, URDF)
Before this commit: robot IRB1100_4kg_580_STD, 7 links, 6 joints
Links:
- removed link link_1_1
- removed link link_2_1
- removed link link_3_1
- removed link link_4_1
- removed link link_5_1
- removed link link_6_1
- added link flange
- added link link_1, mass 24.887771906712818; collision mesh filename=meshes/link_1.stl scale=0.001 0.001 0.001; visual mesh filename=meshes/link_1.stl scale=0.001 0.001 0.001
- added link link_2, mass 19.747227512978796; collision mesh filename=meshes/link_2.stl scale=0.001 0.001 0.001; visual mesh filename=meshes/link_2.stl scale=0.001 0.001 0.001
- added link link_3, mass 8.184213468997186; collision mesh filename=meshes/link_3.stl scale=0.001 0.001 0.001; visual mesh filename=meshes/link_3.stl scale=0.001 0.001 0.001
- added link link_4, mass 12.239054477267983; collision mesh filename=meshes/link_4.stl scale=0.001 0.001 0.001; visual mesh filename=meshes/link_4.stl scale=0.001 0.001 0.001
- added link link_5, mass 2.582057522638694; collision mesh filename=meshes/link_5.stl scale=0.001 0.001 0.001; visual mesh filename=meshes/link_5.stl scale=0.001 0.001 0.001
- added link link_6, mass 0.05751158667684081; collision mesh filename=meshes/link_6.stl scale=0.001 0.001 0.001; visual mesh filename=meshes/link_6.stl scale=0.001 0.001 0.001
- added link tool0
Joints:
- removed joint j1
- removed joint j2
- removed joint j3
- removed joint j4
- removed joint j5
- removed joint j6
- added joint flange-tool0: type fixed, parent flange, child tool0, origin xyz=0.0 0.0 0.0 rpy=0 0 0
- added joint joint_1: type revolute, parent base_link, child link_1, origin xyz=0.0 0.0 0.146 rpy=0 0 0, axis 0.0 0.0 1.0, limit lower=-4.014 upper=4.014 effort=0.0 velocity=8.03
- added joint joint_2: type revolute, parent link_1, child link_2, origin xyz=0.0 0.046 0.181 rpy=0 0 0, axis 0.0 -1.0 -0.0, limit lower=-2.007 upper=1.972 effort=0.0 velocity=6.28
- added joint joint_3: type revolute, parent link_2, child link_3, origin xyz=0.0 0.0026 0.28 rpy=0 0 0, axis 0.0 -1.0 0.0, limit lower=-3.577 upper=0.960 effort=0.0 velocity=4.89
- added joint joint_4: type revolute, parent link_3, child link_4, origin xyz=0.0455 -0.0486 0.01 rpy=0 0 0, axis -1.0 0.0 0.0, limit lower=-4.014 upper=4.014 effort=0.0 velocity=9.77
- added joint joint_5: type revolute, parent link_4, child link_5, origin xyz=0.2545 -0.0325 0.0 rpy=0 0 0, axis -0.0 -1.0 -0.0, limit lower=-2.181 upper=2.094 effort=0.0 velocity=7.33
- added joint joint_6: type revolute, parent link_5, child link_6, origin xyz=0.0634 0.0325 0.0 rpy=0 0 0, axis 1.0 0.0 0.0, limit lower=-6.981 upper=6.981 effort=0.0 velocity=13.09
- added joint joint_6-flange: type fixed, parent link_6, child flange, origin xyz=0.0 0.0 0.0 rpy=0 1.57 0

File: generated/IRB1200H_5_90_STD_v1/IRB1200H_5_90_STD.urdf (robot description, URDF)
Before this commit: robot IRB1200H_5_90_STD, 7 links, 6 joints
Links:
- removed link link_1_1
- removed link link_2_1
- removed link link_3_1
- removed link link_4_1
- removed link link_5_1
- removed link link_6_1
- added link flange
- added link link_1, mass 47.66891611618349; collision mesh filename=meshes/link_1.stl scale=0.001 0.001 0.001; visual mesh filename=meshes/link_1.stl scale=0.001 0.001 0.001
- added link link_2, mass 62.596941650298746; collision mesh filename=meshes/link_2.stl scale=0.001 0.001 0.001; visual mesh filename=meshes/link_2.stl scale=0.001 0.001 0.001
- added link link_3, mass 50.251919251788294; collision mesh filename=meshes/link_3.stl scale=0.001 0.001 0.001; visual mesh filename=meshes/link_3.stl scale=0.001 0.001 0.001
- added link link_4, mass 14.103086555281287; collision mesh filename=meshes/link_4.stl scale=0.001 0.001 0.001; visual mesh filename=meshes/link_4.stl scale=0.001 0.001 0.001
- added link link_5, mass 4.542326712154526; collision mesh filename=meshes/link_5.stl scale=0.001 0.001 0.001; visual mesh filename=meshes/link_5.stl scale=0.001 0.001 0.001
- added link link_6, mass 0.03668180966446797; collision mesh filename=meshes/link_6.stl scale=0.001 0.001 0.001; visual mesh filename=meshes/link_6.stl scale=0.001 0.001 0.001
- added link tool0
Joints:
- removed joint j1
- removed joint j2
- removed joint j3
- removed joint j4
- removed joint j5
- removed joint j6
- added joint flange-tool0: type fixed, parent flange, child tool0, origin xyz=0.0 0.0 0.0 rpy=0 0 0
- added joint joint_1: type revolute, parent base_link, child link_1, origin xyz=0.0 0.0 0.219 rpy=0 0 0, axis 0.0 0.0 -1.0, limit lower=-2.9671 upper=2.9671 effort=0 velocity=5.0265
- added joint joint_2: type revolute, parent link_1, child link_2, origin xyz=0.0 0.06 0.1801 rpy=0 0 0, axis 0.0 -1.0 0.0, limit lower=-1.7453 upper=2.2689 effort=0 velocity=3.9095
- added joint joint_3: type revolute, parent link_2, child link_3, origin xyz=0.0 0.004 0.448 rpy=0 0 0, axis 0.0 -1.0 0.0, limit lower=-3.4907 upper=1.2217 effort=0 velocity=5.1836
- added joint joint_4: type revolute, parent link_3, child link_4, origin xyz=0.2885 -0.064 0.041489 rpy=0 0 0, axis 1.0 0.0 0.0, limit lower=-4.7124 upper=4.7124 effort=0 velocity=6.9813
- added joint joint_5: type revolute, parent link_4, child link_5, origin xyz=0.162491 0.0255 0.000511 rpy=0 0 0, axis 0.0 -1.0 0.0, limit lower=-2.2689 upper=2.2689 effort=0 velocity=7.0686
- added joint joint_6: type revolute, parent link_5, child link_6, origin xyz=0.085509 -0.025514 1.2e-05 rpy=0 0 0, axis 1.0 0.0 0.0, limit lower=-6.9813 upper=6.9813 effort=0 velocity=10.4719
- added joint joint_6-flange: type fixed, parent link_6, child flange, origin xyz=0.0 0.0 0.0 rpy=0 1.57 0

File: generated/IRB1200H_7_70_STD_v1/IRB1200H_7_70_STD.urdf (robot description, URDF)
Before this commit: robot IRB1200H_7_70_STD, 7 links, 6 joints
Links:
- removed link link_1_1
- removed link link_2_1
- removed link link_3_1
- removed link link_4_1
- removed link link_5_1
- removed link link_6_1
- added link flange
- added link link_1, mass 47.62183211112662; collision mesh filename=meshes/link_1.stl scale=0.001 0.001 0.001; visual mesh filename=meshes/link_1.stl scale=0.001 0.001 0.001
- added link link_2, mass 54.93093636945645; collision mesh filename=meshes/link_2.stl scale=0.001 0.001 0.001; visual mesh filename=meshes/link_2.stl scale=0.001 0.001 0.001
- added link link_3, mass 38.854634298936446; collision mesh filename=meshes/link_3.stl scale=0.001 0.001 0.001; visual mesh filename=meshes/link_3.stl scale=0.001 0.001 0.001
- added link link_4, mass 14.103514853516494; collision mesh filename=meshes/link_4.stl scale=0.001 0.001 0.001; visual mesh filename=meshes/link_4.stl scale=0.001 0.001 0.001
- added link link_5, mass 4.542326346976594; collision mesh filename=meshes/link_5.stl scale=0.001 0.001 0.001; visual mesh filename=meshes/link_5.stl scale=0.001 0.001 0.001
- added link link_6, mass 0.036681809664465305; collision mesh filename=meshes/link_6.stl scale=0.001 0.001 0.001; visual mesh filename=meshes/link_6.stl scale=0.001 0.001 0.001
- added link tool0
Joints:
- removed joint j1
- removed joint j2
- removed joint j3
- removed joint j4
- removed joint j5
- removed joint j6
- added joint flange-tool0: type fixed, parent flange, child tool0, origin xyz=0 0 0 rpy=0 0 0
- added joint joint_1: type revolute, parent base_link, child link_1, origin xyz=0.0 0.0 0.219 rpy=0 0 0, axis 0.0 0.0 1.0, limit lower=-2.9671 upper=2.9671 effort=0 velocity=5.0265
- added joint joint_2: type revolute, parent link_1, child link_2, origin xyz=0.0 -0.0615 0.1801 rpy=0 0 0, axis 0.0 -1.0 0.0, limit lower=-1.7453 upper=2.2689 effort=0 velocity=3.9095
- added joint joint_3: type revolute, parent link_2, child link_3, origin xyz=0.0 0.0005 0.35 rpy=0 0 0, axis 0.0 -1.0 0.0, limit lower=-3.4907 upper=1.2217 effort=0 velocity=5.1836
- added joint joint_4: type revolute, parent link_3, child link_4, origin xyz=0.1655 0.06088 0.041999 rpy=0 0 0, axis -1.0 0.0 1.7e-05, limit lower=-4.7124 upper=4.7124 effort=0 velocity=6.9813
- added joint joint_5: type revolute, parent link_4, child link_5, origin xyz=0.1855 0.025499 1e-06 rpy=0 0 0, axis 0.0 -1.0 0.0, limit lower=-2.2689 upper=2.2689 effort=0 velocity=7.0686
- added joint joint_6: type revolute, parent link_5, child link_6, origin xyz=0.0855 -0.025383 0.0 rpy=0 0 0, axis 1.0 0.0 0.0, limit lower=-6.9813 upper=6.9813 effort=0 velocity=10.4719
- added joint joint_6-flange: type fixed, parent link_6, child flange, origin xyz=0 0 0 rpy=0 1.57 0
