Commit message: Validation, limits, and robot improvements
- Add joint limits to all robot models
- Standardize mesh naming conventions (link_1, link_2, etc.)
- Fix joint limits and axis orientations
- Add URDF validation tool
- Update README with robot table and validation info
- Add IK demo scripts and utilities
- Improve documentation and project structure

🤖 Generated with [Claude Code](https://claude.ai/code)

Co-Authored-By: Claude <noreply@anthropic.com>

File: generated/IRB1200_5_90_STD_v1/IRB1200_5_90_STD.urdf (robot description, URDF)
Before this commit: robot IRB1200_5_90_STD, 7 links, 6 joints
Links:
- removed link link_1_1
- removed link link_2_1
- removed link link_3_1
- removed link link_4_1
- removed link link_5_1
- removed link link_6_1
- added link flange, mass 0.01
- added link link_1, mass 47.59365241562889; collision mesh filename=meshes/link_1.stl scale=0.001 0.001 0.001; visual mesh filename=meshes/link_1.stl scale=0.001 0.001 0.001
- added link link_2, mass 0.0002346193667311735; collision mesh filename=meshes/link_2.stl scale=0.001 0.001 0.001; visual mesh filename=meshes/link_2.stl scale=0.001 0.001 0.001
- added link link_3, mass 50.4799691302992; collision mesh filename=meshes/link_3.stl scale=0.001 0.001 0.001; visual mesh filename=meshes/link_3.stl scale=0.001 0.001 0.001
- added link link_4, mass 13.07948314741883; collision mesh filename=meshes/link_4.stl scale=0.001 0.001 0.001; visual mesh filename=meshes/link_4.stl scale=0.001 0.001 0.001
- added link link_5, mass 4.044605310431727; collision mesh filename=meshes/link_5.stl scale=0.001 0.001 0.001; visual mesh filename=meshes/link_5.stl scale=0.001 0.001 0.001
- added link link_6, mass 0.03376885335108457; collision mesh filename=meshes/link_6.stl scale=0.001 0.001 0.001; visual mesh filename=meshes/link_6.stl scale=0.001 0.001 0.001
- added link tool0, mass 0.01
Joints:
- removed joint Revolute_1
- removed joint Revolute_2
- removed joint Revolute_3
- removed joint Revolute_4
- removed joint Revolute_5
- removed joint Revolute_6
- added joint flange-tool0: type fixed, parent flange, child tool0, origin xyz=0 0 0 rpy=0 0 0
- added joint joint_1: type revolute, parent base_link, child link_1, origin xyz=0.0 0.0 0.219 rpy=0 0 0, axis 0.0 0.0 1.0, limit lower=-2.9671 upper=2.9671 effort=0 velocity=5.0265
- added joint joint_2: type revolute, parent link_1, child link_2, origin xyz=0.0 -0.0605 0.1801 rpy=0 0 0, axis 0.0 1.0 0.0, limit lower=-1.7453 upper=2.2689 effort=0 velocity=3.9095
- added joint joint_3: type revolute, parent link_2, child link_3, origin xyz=0.0 0.0025 0.448 rpy=0 0 0, axis 0.0 -1.0 0.0, limit lower=-3.4907 upper=1.2217 effort=0 velocity=5.1836
- added joint joint_4: type revolute, parent link_3, child link_4, origin xyz=0.2885 0.058 0.042 rpy=0 0 0, axis -1.0 0.0 0.0, limit lower=-4.7124 upper=4.7124 effort=0 velocity=6.9813
- added joint joint_5: type revolute, parent link_4, child link_5, origin xyz=0.1625 -0.0285 0.0 rpy=0 0 0, axis 0.0 1.0 0.0, limit lower=-2.2689 upper=2.2689 effort=0 velocity=7.0686
- added joint joint_6: type revolute, parent link_5, child link_6, origin xyz=0.077 0.0285 0.0 rpy=0 0 0, axis 1.0 0.0 0.0, limit lower=-6.9813 upper=6.9813 effort=0 velocity=10.4719
- added joint joint_6-flange: type fixed, parent link_6, child flange, origin xyz=0.005 0 0 rpy=0 1.57 0

File: generated/IRB52_7-1_2-Short_v1/IRB52_7-1_2-Short.urdf (robot description, URDF)
Before this commit: robot IRB52_7_1_2_Short, 7 links, 6 joints
Links:
- added link flange, mass 0.1
- added link tool0, mass 0.01
Joints:
- added joint joint_flange: type fixed, parent link_6, child flange, origin xyz=0 0 0 rpy=0 0 0
- added joint joint_tool0: type fixed, parent flange, child tool0, origin xyz=0 0 0 rpy=0 0 0
- joint joint_1: limit (none) -> lower=-3.14159 upper=3.14159 effort=300 velocity=3.142; type continuous -> revolute
- joint joint_2: limit (none) -> lower=-1.099 upper=1.919 effort=300 velocity=3.142; type continuous -> revolute
- joint joint_3: limit (none) -> lower=-4.101 upper=0.96 effort=300 velocity=3.142; type continuous -> revolute
- joint joint_4: limit (none) -> lower=-3.491 upper=3.491 effort=100 velocity=5.585; type continuous -> revolute
- joint joint_5: limit (none) -> lower=-2.007 upper=2.007 effort=100 velocity=6.981; type continuous -> revolute
- joint joint_6: limit (none) -> lower=-6.981 upper=6.981 effort=100 velocity=8.028; type continuous -> revolute

File: generated/IRB8700_550-420-SW6_v1/IRB8700_550-420-SW6.urdf (robot description, URDF)
Before this commit: robot IRB8700_550_420_SW6, 7 links, 6 joints
Links:
- removed link IRB8700_SW6_550_420_IRC5_rev00_LINK1_CAD_v1_1
- removed link IRB8700_SW6_550_420_IRC5_rev00_LINK2_CAD_v1_1
- removed link IRB8700_SW6_550_420_IRC5_rev00_LINK3_CAD_v1_1
- removed link IRB8700_SW6_550_420_IRC5_rev00_LINK4_CAD_v1_1
- removed link IRB8700_SW6_550_420_IRC5_rev00_LINK5_CAD_v1_1
- removed link IRB8700_SW6_550_420_IRC5_rev00_LINK6_CAD_v1_1
- added link flange, mass 0.1
- added link link_1, mass 1785.9186850506833; collision mesh filename=meshes/link_1.stl scale=0.001 0.001 0.001; visual mesh filename=meshes/link_1.stl scale=0.001 0.001 0.001
- added link link_2, mass 1443.4541146557397; collision mesh filename=meshes/link_2.stl scale=0.001 0.001 0.001; visual mesh filename=meshes/link_2.stl scale=0.001 0.001 0.001
- added link link_3, mass 867.5203145831158; collision mesh filename=meshes/link_3.stl scale=0.001 0.001 0.001; visual mesh filename=meshes/link_3.stl scale=0.001 0.001 0.001
- added link link_4, mass 1308.380613271277; collision mesh filename=meshes/link_4.stl scale=0.001 0.001 0.001; visual mesh filename=meshes/link_4.stl scale=0.001 0.001 0.001
- added link link_5, mass 168.28947433118324; collision mesh filename=meshes/link_5.stl scale=0.001 0.001 0.001; visual mesh filename=meshes/link_5.stl scale=0.001 0.001 0.001
- added link link_6, mass 58.82091127859069; collision mesh filename=meshes/link_6.stl scale=0.001 0.001 0.001; visual mesh filename=meshes/link_6.stl scale=0.001 0.001 0.001
- added link tool0, mass 0.01
Joints:
- removed joint j1
- removed joint j2
- removed joint j3
- removed joint j4
- removed joint j5
- removed joint j6
- added joint joint_1: type revolute, parent base_link, child link_1, origin xyz=0.0 0.0 0.300337 rpy=0 0 0, axis 0.0 -0.0 -1.0, limit lower=-3.839 upper=3.839 effort=100 velocity=1.31
- added joint joint_2: type revolute, parent link_1, child link_2, origin xyz=0.42 0.207 0.699663 rpy=0 0 0, axis 0.0 1.0 0.0, limit lower=-1.134 upper=1.571 effort=80 velocity=1.05
- added joint joint_3: type revolute, parent link_2, child link_3, origin xyz=0.0 0.156 1.58 rpy=0 0 0, axis 0.0 1.0 0.0, limit lower=-0.524 upper=2.303 effort=80 velocity=1.05
- added joint joint_4: type revolute, parent link_3, child link_4, origin xyz=0.344558 -0.363 0.31 rpy=0 0 0, axis 1.0 0.0 0.0, limit lower=-5.236 upper=5.236 effort=60 velocity=1.48
- added joint joint_5: type revolute, parent link_4, child link_5, origin xyz=1.830442 0.145 0.0 rpy=0 0 0, axis 0.0 -1.0 0.0, limit lower=-2.268 upper=2.268 effort=60 velocity=1.48
- added joint joint_6: type revolute, parent link_5, child link_6, origin xyz=0.2605 -0.145 0.0 rpy=0 0 0, axis 1.0 0.0 0.0, limit lower=-6.283 upper=6.283 effort=40 velocity=2.01
- added joint joint_flange: type fixed, parent link_6, child flange, origin xyz=0 0 0 rpy=0 1.57 0
- added joint joint_tool0: type fixed, parent flange, child tool0, origin xyz=0 0 0 rpy=0 0 0

File: generated/IRB8700_800_350_v1/IRB8700_800_350.urdf (robot description, URDF)
Before this commit: robot IRB8700_800_350, 8 links, 7 joints
Links:
- removed link LINK1
- removed link LINK2
- removed link LINK3
- removed link LINK4
- removed link LINK5
- removed link LINK6
- removed link LINKARM
- added link flange, mass 0.1
- added link link_1, mass 1785.9186850506833; collision mesh filename=meshes/link_1.stl scale=0.001 0.001 0.001; visual mesh filename=meshes/link_1.stl scale=0.001 0.001 0.001
- added link link_2, mass 1443.4541146557397; collision mesh filename=meshes/link_2.stl scale=0.001 0.001 0.001; visual mesh filename=meshes/link_2.stl scale=0.001 0.001 0.001
- added link link_3, mass 867.5203145831158; collision mesh filename=meshes/link_3.stl scale=0.001 0.001 0.001; visual mesh filename=meshes/link_3.stl scale=0.001 0.001 0.001
- added link link_4, mass 1084.7317720031733; collision mesh filename=meshes/link_4.stl scale=0.001 0.001 0.001; visual mesh filename=meshes/link_4.stl scale=0.001 0.001 0.001
- added link link_5, mass 180.47343892140714; collision mesh filename=meshes/link_5.stl scale=0.001 0.001 0.001; visual mesh filename=meshes/link_5.stl scale=0.001 0.001 0.001
- added link link_6, mass 24.42929785915679; collision mesh filename=meshes/flange.stl scale=0.001 0.001 0.001; visual mesh filename=meshes/flange.stl scale=0.001 0.001 0.001
- added link tool0, mass 0.01
Joints:
- removed joint j1
- removed joint j2
- removed joint j3
- removed joint j4
- removed joint j5
- removed joint j6
- removed joint tail
- added joint joint_1: type continuous, parent base_link, child link_1, origin xyz=0.0 0.0 0.300337 rpy=0 0 0, axis 0.0 -0.0 -1.0
- added joint joint_2: type continuous, parent link_1, child link_2, origin xyz=0.42 -0.21 0.699663 rpy=0 0 0, axis 0.0 -1.0 0.0
- added joint joint_3: type continuous, parent link_2, child link_3, origin xyz=0.0 -0.153 1.58 rpy=0 0 0, axis 0.0 -1.0 0.0
- added joint joint_4: type continuous, parent link_3, child link_4, origin xyz=0.344558 0.363 0.31 rpy=0 0 0, axis -1.0 0.0 0.0
- added joint joint_5: type continuous, parent link_4, child link_5, origin xyz=1.130442 0.150019 0.000533 rpy=0 0 0, axis 0.0 -0.999391 0.034899
- added joint joint_6: type continuous, parent link_5, child link_6, origin xyz=0.2605 -0.150019 -0.000533 rpy=0 0 0, axis 1.0 0.0 -0.0
- added joint joint_flange: type fixed, parent link_6, child flange, origin xyz=0 0 0 rpy=0 1.57 0
- added joint joint_tool0: type fixed, parent flange, child tool0, origin xyz=0 0 0 rpy=0 0 0

File: generated/IRB920T_6kg_450_180_STD_v1/IRB920T_6kg_450_180_STD.urdf (robot description, URDF)
Before this commit: robot IRB920T_6kg_450_180_STD, 4 links, 3 joints
Links:
- removed link IRB920T_6kg_450_180_STD_OmniCore_rev00_LINK1_CAD_1
- removed link IRB920T_6kg_450_180_STD_OmniCore_rev00_LINK2_CAD_1
- removed link IRB920T_6kg_450_180_STD_OmniCore_rev00_LINK3_CAD_1
- added link flange, mass 0.1
- added link link_1, mass 25.677563367507343; collision mesh filename=meshes/link_1.stl scale=0.001 0.001 0.001; visual mesh filename=meshes/link_1.stl scale=0.001 0.001 0.001
- added link link_2, mass 75.7740500377449; collision mesh filename=meshes/link_2.stl scale=0.001 0.001 0.001; visual mesh filename=meshes/link_2.stl scale=0.001 0.001 0.001
- added link link_3, mass 0.6594614836495646; collision mesh filename=meshes/link_3.stl scale=0.001 0.001 0.001; visual mesh filename=meshes/link_3.stl scale=0.001 0.001 0.001
- added link tool0, mass 0.1
Joints:
- removed joint Revolute_1
- removed joint Revolute_2
- removed joint Slider_3
- added joint joint_1: type continuous, parent base_link, child link_1, origin xyz=-0.00025 2e-06 0.1914 rpy=0 0 0, axis 0.0 0.0 1.0, limit lower=-2.61799 upper=2.61799 effort=0.0 velocity=0.0
- added joint joint_2: type continuous, parent link_1, child link_2, origin xyz=0.191748 -2e-06 0.0871 rpy=0 0 0, axis 0.0 0.0 1.0, limit lower=-2.53073 upper=2.53073 effort=0.0 velocity=0.0
- added joint joint_3: type prismatic, parent link_2, child link_3, origin xyz=0.258502 -0.0 0.305 rpy=0 0 0, axis 0.0 0.0 1.0, limit lower=0.0 upper=0.145 effort=0.0 velocity=0.0
- added joint joint_4: type continuous, parent link_3, child flange, origin xyz=0 0 0 rpy=0 0 0, axis 0.0 0.0 1.0, limit lower=-6.98132 upper=6.98132 effort=0.0 velocity=0.0
- added joint joint_tool0: type fixed, parent flange, child tool0, origin xyz=0.0 0.0 0.0 rpy=0 0 0

File: generated/IRB920_6kg-550-180-STD_v1/IRB920_6kg_550_180_STD.urdf (robot description, URDF)
Before this commit: robot IRB920_6kg_550_180_STD, 4 links, 3 joints
Links:
- removed link link1_1
- removed link link2_1
- removed link link3_1
- added link flange, mass 0.1
- added link link_1, mass 32.62635723576266; collision mesh filename=meshes/link_1.stl scale=0.001 0.001 0.001; visual mesh filename=meshes/link_1.stl scale=0.001 0.001 0.001
- added link link_2, mass 75.77408460894007; collision mesh filename=meshes/link_2.stl scale=0.001 0.001 0.001; visual mesh filename=meshes/link_2.stl scale=0.001 0.001 0.001
- added link link_3, mass 0.6594614836495646; collision mesh filename=meshes/link_3.stl scale=0.001 0.001 0.001; visual mesh filename=meshes/link_3.stl scale=0.001 0.001 0.001
- added link tool0, mass 0.1
Joints:
- removed joint j1
- removed joint j2
- removed joint j3
- added joint joint_1: type continuous, parent base_link, child link_1, origin xyz=-0.027677 -0.027437 0.1914 rpy=0 0 0, axis 0.0 0.0 1.0, limit lower=-2.61799 upper=2.61799 effort=0.0 velocity=0.0
- added joint joint_2: type continuous, parent link_1, child link_2, origin xyz=0.0 -0.29 0.086 rpy=0 0 0, axis 0.0 0.0 1.0, limit lower=-2.53073 upper=2.53073 effort=0.0 velocity=0.0
- added joint joint_3: type prismatic, parent link_2, child link_3, origin xyz=0.0 -0.26 -0.036 rpy=0 0 0, axis -0.0 -0.0 -1.0, limit lower=0.0 upper=0.145 effort=0.0 velocity=0.0
- added joint joint_4: type continuous, parent link_3, child flange, origin xyz=0 0 0 rpy=0 0 0, axis 0.0 0.0 1.0, limit lower=-6.98132 upper=6.98132 effort=0.0 velocity=0.0
- added joint joint_tool0: type fixed, parent flange, child tool0, origin xyz=0.0 0.0 0.0 rpy=0 0 0

File: generated/IRB920_6kg_650_180_STD_v1/IRB920_6kg_650_180_STD.urdf (robot description, URDF)
Before this commit: robot IRB920_6kg_650_180_STD, 4 links, 3 joints
Links:
- removed link IRB920_6kg_650_180_STD_OmniCore_rev00_LINK1_CAD_STEP_1
- removed link IRB920_6kg_650_180_STD_OmniCore_rev00_LINK2_CAD_STEP_1
- removed link IRB920_6kg_650_180_STD_OmniCore_rev00_LINK3_CAD_STEP_1
- added link flange, mass 0.1
- added link link_1, mass 40.4824375073; collision mesh filename=meshes/link_1.stl scale=0.001 0.001 0.001; visual mesh filename=meshes/link_1.stl scale=0.001 0.001 0.001
- added link link_2, mass 75.77408460831636; collision mesh filename=meshes/link_2.stl scale=0.001 0.001 0.001; visual mesh filename=meshes/link_2.stl scale=0.001 0.001 0.001
- added link link_3, mass 0.6594614836495672; collision mesh filename=meshes/link_3.stl scale=0.001 0.001 0.001; visual mesh filename=meshes/link_3.stl scale=0.001 0.001 0.001
- added link tool0, mass 0.01
Joints:
- removed joint Revolute_1
- removed joint Revolute_2
- removed joint Slider_3
- added joint joint_1: type revolute, parent base_link, child link_1, origin xyz=-0.00025 2e-06 0.1914 rpy=0 0 0, axis 0.0 0.0 1.0, limit lower=-2.61799 upper=2.61799 effort=0.0 velocity=0.0
- added joint joint_2: type revolute, parent link_1, child link_2, origin xyz=0.391748 -2e-06 0.0871 rpy=0 0 0, axis 0.0 0.0 1.0, limit lower=-2.53073 upper=2.53073 effort=0.0 velocity=0.0
- added joint joint_3: type prismatic, parent link_2, child link_3, origin xyz=0.258502 -0.0 0.305 rpy=0 0 0, axis 0.0 0.0 1.0, limit lower=0.0 upper=0.145 effort=0.0 velocity=0.0
- added joint joint_4: type revolute, parent link_3, child flange, origin xyz=0 0 0 rpy=0 0 0, axis 0.0 0.0 1.0, limit lower=-6.98132 upper=6.98132 effort=0.0 velocity=0.0
- added joint joint_tool0: type fixed, parent flange, child tool0, origin xyz=0 0 0 rpy=0 0 0

File: generated/IRB930_12kg_1050_300_STD_v1/IRB930_12kg_1050_300_STD.urdf (robot description, URDF)
Before this commit: robot IRB930_12kg_1050_300_STD_Omnicore_rev00_Assembly, 4 links, 3 joints
Links:
- removed link IRB930_12kg_1050_300_STD_Omnicore_rev00_LINK1_CAD_1
- removed link IRB930_12kg_1050_300_STD_Omnicore_rev00_LINK2_CAD_1
- removed link IRB930_12kg_1050_300_STD_Omnicore_rev00_LINK3_CAD_1
- added link flange, mass 0.1
- added link link_1, mass 104.004672609044; collision mesh filename=meshes/link_1.stl scale=0.001 0.001 0.001; visual mesh filename=meshes/link_1.stl scale=0.001 0.001 0.001
- added link link_2, mass 199.4580874558294; collision mesh filename=meshes/link_2.stl scale=0.001 0.001 0.001; visual mesh filename=meshes/link_2.stl scale=0.001 0.001 0.001
- added link link_3, mass 1.6450553674720612; collision mesh filename=meshes/link_3.stl scale=0.001 0.001 0.001; visual mesh filename=meshes/link_3.stl scale=0.001 0.001 0.001
- added link tool0, mass 0.1
Joints:
- removed joint Revolute_1
- removed joint Revolute_2
- removed joint Slider_3
- added joint joint_1: type continuous, parent base_link, child link_1, origin xyz=0.0 0.0 0.272 rpy=0 0 0, axis 0.0 0.0 1.0
- added joint joint_2: type continuous, parent link_1, child link_2, origin xyz=0.56 0.0 0.1235 rpy=0 0 0, axis 0.0 0.0 1.0
- added joint joint_3: type prismatic, parent link_2, child link_3, origin xyz=0.49 0.0 0.1687 rpy=0 0 0, axis -0.0 0.0 1.0, limit lower=-0.2 upper=0.0 effort=100 velocity=100
- added joint joint_4: type continuous, parent link_3, child flange, origin xyz=0 0 0 rpy=0 0 0, axis 0.0 0.0 1.0, limit lower=-6.98132 upper=6.98132 effort=0.0 velocity=0.0
- added joint joint_tool0: type fixed, parent flange, child tool0, origin xyz=0.0 0.0 0.0 rpy=0 0 0
