Commit message: regen all usd files

File: library/ABB/IRB14050_SAYuMi_v1/IRB14050_SAYuMi.urdf (robot description, URDF)
Before this commit: robot IRB14050_SAYuMi, 8 links, 7 joints
Links:
- removed link Link1_R_1
- removed link Link2_R_1
- removed link Link3_R_1
- removed link Link4_R_1
- removed link Link5_R_1
- removed link Link6_R_1
- removed link Link7_R_1
- added link flange, mass 0.1
- added link link_1, mass 7.562885567589252; collision mesh filename=meshes/link_1.stl scale=0.001 0.001 0.001; visual mesh filename=meshes/link_1.stl scale=0.001 0.001 0.001
- added link link_2, mass 11.070792495652707; collision mesh filename=meshes/link_2.stl scale=0.001 0.001 0.001; visual mesh filename=meshes/link_2.stl scale=0.001 0.001 0.001
- added link link_3, mass 6.048580949750527; collision mesh filename=meshes/link_3.stl scale=0.001 0.001 0.001; visual mesh filename=meshes/link_3.stl scale=0.001 0.001 0.001
- added link link_4, mass 9.26921022899374; collision mesh filename=meshes/link_4.stl scale=0.001 0.001 0.001; visual mesh filename=meshes/link_4.stl scale=0.001 0.001 0.001
- added link link_5, mass 2.6959499165850227; collision mesh filename=meshes/link_5.stl scale=0.001 0.001 0.001; visual mesh filename=meshes/link_5.stl scale=0.001 0.001 0.001
- added link link_6, mass 3.6915533716806794; collision mesh filename=meshes/link_6.stl scale=0.001 0.001 0.001; visual mesh filename=meshes/link_6.stl scale=0.001 0.001 0.001
- added link link_7, mass 0.240688664570473; collision mesh filename=meshes/link_7.stl scale=0.001 0.001 0.001; visual mesh filename=meshes/link_7.stl scale=0.001 0.001 0.001
- added link tool0, mass 0.01
Joints:
- removed joint j1
- removed joint j2
- removed joint j3
- removed joint j4
- removed joint j5
- removed joint j6
- removed joint j7
- added joint joint_1: type revolute, parent base_link, child link_1, origin xyz=0.0 0.0 0.173832 rpy=0 0 0, axis 0.0 0.0 -1.0, limit lower=-2.967 upper=2.967 effort=50 velocity=2.618
- added joint joint_2: type revolute, parent link_1, child link_2, origin xyz=-0.03 0.012 0.132 rpy=0 0 0, axis 0.0 1.0 0.0, limit lower=-2.269 upper=0.759 effort=50 velocity=2.618
- added joint joint_3: type revolute, parent link_2, child link_3, origin xyz=0.03 -0.011 0.17283 rpy=0 0 0, axis -0.0 -0.0 1.0, limit lower=-2.967 upper=2.967 effort=50 velocity=2.618
- added joint joint_4: type revolute, parent link_3, child link_4, origin xyz=0.0405 0.011 0.079096 rpy=0 0 0, axis -0.0 -1.0 -0.0, limit lower=-1.396 upper=2.269 effort=50 velocity=2.618
- added joint joint_5: type revolute, parent link_4, child link_5, origin xyz=0.164649 -0.013 0.040333 rpy=0 0 0, axis -0.999999 0.0 0.00101, limit lower=-5.236 upper=5.236 effort=50 velocity=2.618
- added joint joint_6: type revolute, parent link_5, child link_6, origin xyz=0.100365 0.027012 -0.027089 rpy=0 0 0, axis 0.0 1.0 0.000441, limit lower=-1.571 upper=2.094 effort=50 velocity=2.618
- added joint joint_7: type revolute, parent link_6, child link_7, origin xyz=0.024836 -0.027012 0.027139 rpy=0 0 0, axis -0.999982 3e-06 -0.00607, limit lower=-3.491 upper=3.491 effort=50 velocity=2.618
- added joint joint_flange: type fixed, parent link_7, child flange, origin xyz=0 0 0 rpy=0 1.57 0
- added joint joint_tool0: type fixed, parent flange, child tool0, origin xyz=0 0 0 rpy=0 0 0

File: library/ABB/IRB1520ID_4_150_v1/IRB1520ID_4_150.urdf (robot description, URDF)
Before this commit: robot IRB1520ID_4_150, 9 links, 8 joints
Joints:
- joint joint_6-flange: origin xyz=0.0 0.0 0.0 rpy=0 0 0 -> xyz=0.0 0.0 0.0 rpy=0 1.57 0

File: library/ABB/IRB1600_X-120_v1/IRB1600_X-120.urdf (robot description, URDF)
Before this commit: robot IRB1600_X_120, 8 links, 7 joints
Joints:
- joint joint_6: origin xyz=-0.032999 0.0245 0.0 rpy=0 0 0 -> xyz=-0.032999 0.0245 0.0 rpy=0 1.57 0

File: library/ABB/IRB52_7-1_2-Short_v1/IRB52_7-1_2-Short.urdf (robot description, URDF)
Before this commit: robot IRB52_7_1_2_Short, 9 links, 8 joints
Joints:
- joint joint_flange: origin xyz=0 0 0 rpy=0 0 0 -> xyz=0 0 0 rpy=0 1.57 0

File: library/ABB/IRB52_7-1_45-Long_v1/IRB52_7-1_45-Long.urdf (robot description, URDF)
Before this commit: robot IRB52_7_1_45_Long, 9 links, 8 joints
Joints:
- joint joint_6-flange: origin xyz=0.0 0.0 0.0 rpy=0 0 0 -> xyz=0.0 0.0 0.0 rpy=0 1.57 0

File: library/ABB/IRB5500-22_v1/IRB5500-22.urdf (robot description, URDF)
Before this commit: robot IRB5500_22, 10 links, 9 joints
Joints:
- joint joint_6_flange: origin xyz=0 0 0 rpy=0 0 0 -> xyz=0 0 0 rpy=0 1.57 0

File: library/ABB/IRB5500-27_v1/IRB5500-27.urdf (robot description, URDF)
Before this commit: robot IRB5500_27_rev00, 10 links, 9 joints
Joints:
- joint joint_6-flange: origin xyz=0.03659 0.013541 -0.066378 rpy=0 0 0 -> xyz=0.03659 0.013541 -0.066378 rpy=0 1.57 0

File: library/ABB/IRB5510-12_v1/IRB5510-12.urdf (robot description, URDF)
Before this commit: robot IRB5510_12, 9 links, 8 joints
Joints:
- joint joint_6b: origin xyz=0.086813 0.003441 0.0 rpy=0 0 0 -> xyz=0.086813 0.003441 0.0 rpy=0 1.57 0

File: library/ABB/IRB6750S_185-390-LID_v1/IRB6750S_185-390-LID.urdf (robot description, URDF)
Before this commit: robot IRB6750S_185_390_LID, 10 links, 9 joints
Joints:
- joint link_6_to_flange: origin xyz=0 0 0 rpy=0 0 0 -> xyz=0 0 0 rpy=0 1.57 0
