Commit message: URDF Refinements (missing limits, wrong flange frames etc) (#6)

File: library/ABB/IRB1520ID_4_150_v1/IRB1520ID_4_150.urdf (robot description, URDF)
Before this commit: robot IRB1520ID_4_150, 7 links, 6 joints
Links:
- removed link link_1_1
- removed link link_2_1
- removed link link_3_1
- removed link link_4_1
- removed link link_5_1
- removed link link_6_1
- added link flange
- added link link_1, mass 140.431105262512; collision mesh filename=meshes/link_1.stl scale=0.001 0.001 0.001; visual mesh filename=meshes/link_1.stl scale=0.001 0.001 0.001
- added link link_2, mass 41.09408994963129; collision mesh filename=meshes/link_2.stl scale=0.001 0.001 0.001; visual mesh filename=meshes/link_2.stl scale=0.001 0.001 0.001
- added link link_3, mass 87.68237861319876; collision mesh filename=meshes/link_3.stl scale=0.001 0.001 0.001; visual mesh filename=meshes/link_3.stl scale=0.001 0.001 0.001
- added link link_4, mass 21.10958519516661; collision mesh filename=meshes/link_4.stl scale=0.001 0.001 0.001; visual mesh filename=meshes/link_4.stl scale=0.001 0.001 0.001
- added link link_5, mass 4.145062543835652; collision mesh filename=meshes/link_5.stl scale=0.001 0.001 0.001; visual mesh filename=meshes/link_5.stl scale=0.001 0.001 0.001
- added link link_6, mass 0.7222246780605773; collision mesh filename=meshes/link_6.stl scale=0.001 0.001 0.001; visual mesh filename=meshes/link_6.stl scale=0.001 0.001 0.001
- added link tool0
Joints:
- removed joint j1
- removed joint j2
- removed joint j3
- removed joint j4
- removed joint j5
- removed joint j6
- added joint flange-tool0: type fixed, parent flange, child tool0, origin xyz=0.0 0.0 0.0 rpy=0 0 0
- added joint joint_1: type revolute, parent base_link, child link_1, origin xyz=0.0 0.0 0.179 rpy=0 0 0, axis -0.0 -0.0 1.0, limit lower=-2.967 upper=2.967 effort=250 velocity=2.2689
- added joint joint_2: type revolute, parent link_1, child link_2, origin xyz=0.16 -0.101 0.274 rpy=0 0 0, axis 0.0 -1.0 -0.0, limit lower=-1.571 upper=2.618 effort=200 velocity=2.4435
- added joint joint_3: type revolute, parent link_2, child link_3, origin xyz=0.0 -0.02 0.59 rpy=0 0 0, axis 0.0 -1.0 -0.0, limit lower=-1.745 upper=1.396 effort=180 velocity=2.4435
- added joint joint_4: type revolute, parent link_3, child link_4, origin xyz=0.217 0.121676 0.2 rpy=0 0 0, axis -1.0 -0.0 0.0, limit lower=-2.705 upper=2.705 effort=100 velocity=5.5851
- added joint joint_5: type revolute, parent link_4, child link_5, origin xyz=0.506 0.051824 0.0 rpy=0 0 0, axis 0.0 -1.0 -0.0, limit lower=-2.356 upper=2.356 effort=80 velocity=6.6323
- added joint joint_6: type revolute, parent link_5, child link_6, origin xyz=0.189629 -0.0525 0.0 rpy=0 0 0, axis 1.0 0.0 0.0, limit lower=-3.491 upper=3.491 effort=50 velocity=8.0285
- added joint joint_6-flange: type fixed, parent link_6, child flange, origin xyz=0.0 0.0 0.0 rpy=0 1.57 0

File: library/ABB/IRB1600_X-120_v1/IRB1600_X-120.urdf (robot description, URDF)
Before this commit: robot IRB1600_X_120, 7 links, 6 joints
Links:
- removed link link1_1
- removed link link2_1
- removed link link3_1
- removed link link4_1
- removed link link5_1
- removed link link6_1
- added link flange, mass 0.27547199791088767; collision mesh filename=meshes/flange.stl scale=0.001 0.001 0.001; visual mesh filename=meshes/flange.stl scale=0.001 0.001 0.001
- added link link_1, mass 314.1495566081902; collision mesh filename=meshes/link_1.stl scale=0.001 0.001 0.001; visual mesh filename=meshes/link_1.stl scale=0.001 0.001 0.001
- added link link_2, mass 62.55263861048576; collision mesh filename=meshes/link_2.stl scale=0.001 0.001 0.001; visual mesh filename=meshes/link_2.stl scale=0.001 0.001 0.001
- added link link_3, mass 129.07256427136392; collision mesh filename=meshes/link_3.stl scale=0.001 0.001 0.001; visual mesh filename=meshes/link_3.stl scale=0.001 0.001 0.001
- added link link_4, mass 22.82263512327022; collision mesh filename=meshes/link_4.stl scale=0.001 0.001 0.001; visual mesh filename=meshes/link_4.stl scale=0.001 0.001 0.001
- added link link_5, mass 1.5097987445956202; collision mesh filename=meshes/link_5.stl scale=0.001 0.001 0.001; visual mesh filename=meshes/link_5.stl scale=0.001 0.001 0.001
- added link tool0
Joints:
- removed joint Revolute_1
- removed joint Revolute_2
- removed joint Revolute_3
- removed joint Revolute_4
- removed joint Revolute_5
- removed joint Revolute_6
- added joint flange_to_tool0: type fixed, parent flange, child tool0, origin xyz=0 0 0 rpy=0 0 0
- added joint joint_1: type revolute, parent base_link, child link_1, origin xyz=0.0 0.0 0.1315 rpy=0 0 0, axis 0.0 0.0 -1.0, limit lower=-3.14159 upper=3.14159 effort=1000 velocity=2.618
- added joint joint_2: type revolute, parent link_1, child link_2, origin xyz=0.15 -0.143 0.355 rpy=0 0 0, axis 0.0 1.0 0.0, limit lower=-1.571 upper=2.094 effort=1000 velocity=2.793
- added joint joint_3: type revolute, parent link_2, child link_3, origin xyz=0.0 0.028 0.475 rpy=0 0 0, axis -0.0 1.0 0.0, limit lower=-4.276 upper=1.134 effort=1000 velocity=2.967
- added joint joint_4: type revolute, parent link_3, child link_4, origin xyz=0.314 0.115002 0.0 rpy=0 0 0, axis 1.0 0.0 0.0, limit lower=-3.491 upper=3.491 effort=500 velocity=5.585
- added joint joint_5: type revolute, parent link_4, child link_5, origin xyz=0.286 -0.0248 0.0 rpy=0 0 0, axis 0.0 -1.0 0.0, limit lower=-2.007 upper=2.007 effort=500 velocity=6.981
- added joint joint_6: type revolute, parent link_5, child flange, origin xyz=-0.032999 0.0245 0.0 rpy=0 1.57 0, axis -1.0 0.0 0.0, limit lower=-6.981 upper=6.981 effort=200 velocity=8.029

File: library/ABB/IRB52_7-1_45-Long_v1/IRB52_7-1_45-Long.urdf (robot description, URDF)
Before this commit: robot IRB52_7_1_45_Long, 7 links, 6 joints
Links:
- removed link link_2_1
- removed link link_3_1
- removed link link_4_1
- removed link link_5_1
- removed link link_6_1
- removed link link_7_1
- added link flange
- added link link_1, mass 477.42257605472827; collision mesh filename=meshes/link_1.stl scale=0.001 0.001 0.001; visual mesh filename=meshes/link_1.stl scale=0.001 0.001 0.001
- added link link_2, mass 81.8083114015255; collision mesh filename=meshes/link_2.stl scale=0.001 0.001 0.001; visual mesh filename=meshes/link_2.stl scale=0.001 0.001 0.001
- added link link_3, mass 137.985170387113; collision mesh filename=meshes/link_3.stl scale=0.001 0.001 0.001; visual mesh filename=meshes/link_3.stl scale=0.001 0.001 0.001
- added link link_4, mass 23.228585050319158; collision mesh filename=meshes/link_4.stl scale=0.001 0.001 0.001; visual mesh filename=meshes/link_4.stl scale=0.001 0.001 0.001
- added link link_5, mass 1.0387285866977907; collision mesh filename=meshes/link_5.stl scale=0.001 0.001 0.001; visual mesh filename=meshes/link_5.stl scale=0.001 0.001 0.001
- added link link_6, mass 0.22926812698528237; collision mesh filename=meshes/link_6.stl scale=0.001 0.001 0.001; visual mesh filename=meshes/link_6.stl scale=0.001 0.001 0.001
- added link tool0
Joints:
- removed joint j1
- removed joint j2
- removed joint j3
- removed joint j4
- removed joint j5
- removed joint j6
- added joint flange-tool0: type fixed, parent flange, child tool0, origin xyz=0.0 0.0 0.0 rpy=0 0 0
- added joint joint_1: type revolute, parent base_link, child link_1, origin xyz=0.0 0.0 0.1245 rpy=0 0 0, axis 0.0 0.0 -1.0, limit lower=-3.14159 upper=3.14159 effort=300 velocity=3.142
- added joint joint_2: type revolute, parent link_1, child link_2, origin xyz=0.15 -0.138 0.362 rpy=0 0 0, axis 0.0 -1.0 0.0, limit lower=-1.099 upper=1.919 effort=300 velocity=3.142
- added joint joint_3: type revolute, parent link_2, child link_3, origin xyz=0.0 0.023 0.7 rpy=0 0 0, axis 0.0 1.0 0.0, limit lower=-4.101 upper=0.96 effort=300 velocity=3.142
- added joint joint_4: type revolute, parent link_3, child link_4, origin xyz=0.314 0.115 0.0 rpy=0 0 0, axis -1.0 0.0 0.0, limit lower=-3.491 upper=3.491 effort=100 velocity=5.585
- added joint joint_5: type revolute, parent link_4, child link_5, origin xyz=0.286 -0.01365 0.0 rpy=0 0 0, axis 0.0 1.0 0.0, limit lower=-2.007 upper=2.007 effort=100 velocity=6.981
- added joint joint_6: type revolute, parent link_5, child link_6, origin xyz=0.042004 0.01365 0.0 rpy=0 0 0, axis 1.0 0.0 0.0, limit lower=-6.981 upper=6.981 effort=100 velocity=8.028
- added joint joint_6-flange: type fixed, parent link_6, child flange, origin xyz=0.0 0.0 0.0 rpy=0 1.57 0

File: library/ABB/IRB5500-22_v1/IRB5500-22.urdf (robot description, URDF)
Before this commit: robot IRB5500_22_rev00, 8 links, 7 joints
Links:
- removed link IRB5500_22_rev00_LINK1_CAD_1
- removed link IRB5500_22_rev00_LINK2_CAD_1
- removed link IRB5500_22_rev00_LINK3_CAD_1
- removed link IRB5500_22_rev00_LINK4_CAD_1
- removed link IRB5500_22_rev00_LINK5B_CAD_1
- removed link IRB5500_22_rev00_LINK5_CAD_1
- removed link IRB5500_22_rev00_LINK6_CAD_1
- added link flange
- added link link_1, mass 1170.5411783269178; collision mesh filename=meshes/link_1.stl scale=0.001 0.001 0.001; visual mesh filename=meshes/link_1.stl scale=0.001 0.001 0.001
- added link link_2, mass 723.6999417469983; collision mesh filename=meshes/link_2.stl scale=0.001 0.001 0.001; visual mesh filename=meshes/link_2.stl scale=0.001 0.001 0.001
- added link link_3, mass 607.3432707370075; collision mesh filename=meshes/link_3.stl scale=0.001 0.001 0.001; visual mesh filename=meshes/link_3.stl scale=0.001 0.001 0.001
- added link link_4, mass 13.246564877496244; collision mesh filename=meshes/link_4.stl scale=0.001 0.001 0.001; visual mesh filename=meshes/link_4.stl scale=0.001 0.001 0.001
- added link link_5, mass 22.90378370207612; collision mesh filename=meshes/link_5.stl scale=0.001 0.001 0.001; visual mesh filename=meshes/link_5.stl scale=0.001 0.001 0.001
- added link link_5b, mass 11.027488801145376; collision mesh filename=meshes/link_5b.stl scale=0.001 0.001 0.001; visual mesh filename=meshes/link_5b.stl scale=0.001 0.001 0.001
- added link link_6, mass 0.3574993425525093; collision mesh filename=meshes/link_6.stl scale=0.001 0.001 0.001; visual mesh filename=meshes/link_6.stl scale=0.001 0.001 0.001
- added link tool0
Joints:
- removed joint j1
- removed joint j2
- removed joint j3
- removed joint j4
- removed joint j5
- removed joint j6
- removed joint j6b
- added joint flange_tool0: type fixed, parent flange, child tool0, origin xyz=0 0 0 rpy=0 0 0
- added joint joint_1: type continuous, parent base_link, child link_1, origin xyz=0.515249 0.226004 0.484024 rpy=0 0 0, axis -0.0 0.000105 -1.0
- added joint joint_2: type continuous, parent link_1, child link_2, origin xyz=0.0 -0.231046 0.435976 rpy=0 0 0, axis -0.0 -1.0 -0.000105
- added joint joint_3: type continuous, parent link_2, child link_3, origin xyz=0.000202 0.035675 1.300003 rpy=0 0 0, axis -0.0 1.0 0.000105
- added joint joint_4: type continuous, parent link_3, child link_4, origin xyz=1.441 0.217 -3.9e-05 rpy=0 0 0, axis 1.0 -0.0 0.0
- added joint joint_5: type continuous, parent link_4, child link_5, origin xyz=0.074415 -0.003442 0.0 rpy=0 0 0, axis 0.819152 -0.573576 -6e-05
- added joint joint_6: type continuous, parent link_5, child link_5b, origin xyz=0.119872 0.0 0.0 rpy=0 0 0, axis 0.819152 0.573576 6e-05
- added joint joint_6_flange: type fixed, parent link_6, child flange, origin xyz=0 0 0 rpy=0 1.57 0
- added joint joint_6b: type revolute, parent link_5b, child link_6, origin xyz=0.086813 0.003442 0.0 rpy=0 0 0, axis -1.0 0.0 -0.0, limit lower=0.0 upper=0.0 effort=100 velocity=100

File: library/ABB/IRB5500-27_v1/IRB5500-27.urdf (robot description, URDF)
Before this commit: robot IRB5500_27_rev00, 9 links, 8 joints
Links:
- removed link IRB5500_27_rev00_AXIS7_ELBOW_CAD_1
- removed link IRB5500_27_rev00_LINK1_CAD_1
- removed link IRB5500_27_rev00_LINK2_CAD_1
- removed link IRB5500_27_rev00_LINK3_CAD_1
- removed link IRB5500_27_rev00_LINK4_CAD_1
- removed link IRB5500_27_rev00_LINK5B_CAD_1
- removed link IRB5500_27_rev00_LINK5_CAD_1
- removed link IRB5500_27_rev00_LINK6_CAD_1
- added link flange, mass 0.3574993425525092; collision mesh filename=meshes/flange.stl scale=0.001 0.001 0.001; visual mesh filename=meshes/flange.stl scale=0.001 0.001 0.001
- added link link_1, mass 702.2698415858004; collision mesh filename=meshes/link_1.stl scale=0.001 0.001 0.001; visual mesh filename=meshes/link_1.stl scale=0.001 0.001 0.001
- added link link_2, mass 1176.3951689098158; collision mesh filename=meshes/link_2.stl scale=0.001 0.001 0.001; visual mesh filename=meshes/link_2.stl scale=0.001 0.001 0.001
- added link link_3, mass 723.6999417468928; collision mesh filename=meshes/link_3.stl scale=0.001 0.001 0.001; visual mesh filename=meshes/link_3.stl scale=0.001 0.001 0.001
- added link link_4, mass 607.3432806136773; collision mesh filename=meshes/link_4.stl scale=0.001 0.001 0.001; visual mesh filename=meshes/link_4.stl scale=0.001 0.001 0.001
- added link link_5, mass 13.246564877496244; collision mesh filename=meshes/link_5.stl scale=0.001 0.001 0.001; visual mesh filename=meshes/link_5.stl scale=0.001 0.001 0.001
- added link link_6, mass 22.90378370207619; collision mesh filename=meshes/link_6.stl scale=0.001 0.001 0.001; visual mesh filename=meshes/link_6.stl scale=0.001 0.001 0.001
- added link link_7, mass 11.0274888011437; collision mesh filename=meshes/link_7.stl scale=0.001 0.001 0.001; visual mesh filename=meshes/link_7.stl scale=0.001 0.001 0.001
- added link tool0
Joints:
- removed joint eoat
- removed joint j1
- removed joint j2
- removed joint j3
- removed joint j4
- removed joint j5
- removed joint j6
- removed joint j7
- added joint flange-tool0: type fixed, parent flange, child tool0, origin xyz=0 0 0 rpy=0 0 0
- added joint joint_1: type continuous, parent base_link, child link_1, origin xyz=0.0 -0.193265 1.160001 rpy=0 0 0, axis 0.0 0.0 1.0
- added joint joint_2: type continuous, parent link_1, child link_2, origin xyz=0.0 0.3975 -0.6285 rpy=0 0 0, axis 0.0 1.0 0.0
- added joint joint_3: type continuous, parent link_2, child link_3, origin xyz=-0.231 0.436 0.0 rpy=0 0 0, axis -1.0 -0.0 -0.0
- added joint joint_4: type continuous, parent link_3, child link_4, origin xyz=0.014 1.3 0.0 rpy=0 0 0, axis 1.0 0.0 -0.0
- added joint joint_5: type continuous, parent link_4, child link_5, origin xyz=0.222 0.0 -1.441 rpy=0 0 0, axis 0.0 -0.0 -1.0
- added joint joint_6: type continuous, parent link_5, child link_6, origin xyz=-0.002653 0.002191 -0.074415 rpy=0 0 0, axis -0.442229 0.365272 -0.819152
- added joint joint_6-flange: type fixed, parent link_7, child flange, origin xyz=0.03659 0.013541 -0.066378 rpy=0 1.57 0, axis -0.4723 -0.219672 0.853626, limit lower=0.0 upper=0.0 effort=100 velocity=100
- added joint joint_7: type continuous, parent link_6, child link_7, origin xyz=-0.000861 -0.001025 -0.119865 rpy=0 0 0, axis 0.430464 -0.379286 -0.81905

File: library/ABB/IRB5510-12_v1/IRB5510-12.urdf (robot description, URDF)
Before this commit: robot IRB5510_12, 8 links, 7 joints
Links:
- removed link link6
- added link flange, mass 0.3574993425525093; collision mesh filename=meshes/flange.stl scale=0.001 0.001 0.001; visual mesh filename=meshes/flange.stl scale=0.001 0.001 0.001
- added link tool0
Joints:
- removed joint joint1
- removed joint joint2
- removed joint joint3
- removed joint joint4
- removed joint joint5
- removed joint joint6
- removed joint joint6b
- added joint flange-tool0: type fixed, parent flange, child tool0, origin xyz=0 0 0 rpy=0 0 0
- added joint joint_1: type revolute, parent base_link, child link1, origin xyz=0.0 0.0 0.484 rpy=0 0 0, axis 0.0 0.0 -1.0, limit lower=-6.283 upper=6.283 effort=0 velocity=1.745
- added joint joint_2: type revolute, parent link1, child link2, origin xyz=-0.0 -0.231 0.436 rpy=0 0 0, axis 0.0 1.0 0.0, limit lower=-6.283 upper=6.283 effort=0 velocity=1.745
- added joint joint_3: type revolute, parent link2, child link3, origin xyz=0.0 0.014 1.1 rpy=0 0 0, axis 0.0 1.0 0.0, limit lower=-6.283 upper=6.283 effort=0 velocity=1.745
- added joint joint_4: type revolute, parent link3, child link4, origin xyz=1.219 0.217 0.0 rpy=0 0 0, axis 1.0 0.0 0.0, limit lower=-1.309 upper=1.309 effort=0 velocity=8.116
- added joint joint_5: type revolute, parent link4, child link5, origin xyz=0.074415 -0.003441 0.0 rpy=0 0 0, axis 0.819152 -0.573576 0.0, limit lower=-1.309 upper=1.309 effort=0 velocity=6.109
- added joint joint_6: type revolute, parent link5, child link5b, origin xyz=0.119872 0.0 0.0 rpy=0 0 0, axis 0.819152 0.573576 0.0, limit lower=-8.029 upper=8.029 effort=0 velocity=9.337
- added joint joint_6b: type revolute, parent link5b, child flange, origin xyz=0.086813 0.003441 0.0 rpy=0 1.57 0, axis -1.0 0.0 -0.0, limit lower=0.0 upper=0.0 effort=100 velocity=100

File: library/ABB/IRB6750S_185-390-LID_v1/IRB6750S_185-390-LID.urdf (robot description, URDF)
Before this commit: robot IRB6750S_185_390_LID, 8 links, 7 joints
Links:
- removed link IRB6750S_All_390_OC_00_LINK04_CAD_v1_1
- removed link IRB6750S_All_390_OC_00_LINK05_CAD_v1_1
- removed link IRB6750S_All_OC_00_CYL_CAD_v1_1
- removed link IRB6750S_All_OC_00_LINK01_CAD_v1_1
- removed link IRB6750S_All_OC_00_LINK02_CAD_v1_1
- removed link IRB6750S_All_OC_00_LINK03_CAD_v1_1
- removed link IRB6750S_LID_185kg_390_OC_00_LINK06_CABLE_v1_1
- added link counter_cylinder, mass 891.4689007968218; collision mesh filename=meshes/counter_cylinder.stl scale=0.001 0.001 0.001; visual mesh filename=meshes/counter_cylinder.stl scale=0.001 0.001 0.001
- added link flange
- added link link_1, mass 855.1080095158879; collision mesh filename=meshes/link_1.stl scale=0.001 0.001 0.001; visual mesh filename=meshes/link_1.stl scale=0.001 0.001 0.001
- added link link_2, mass 745.7860274622177; collision mesh filename=meshes/link_2.stl scale=0.001 0.001 0.001; visual mesh filename=meshes/link_2.stl scale=0.001 0.001 0.001
- added link link_3, mass 497.1042094540328; collision mesh filename=meshes/link_3.stl scale=0.001 0.001 0.001; visual mesh filename=meshes/link_3.stl scale=0.001 0.001 0.001
- added link link_4, mass 593.0820849974; collision mesh filename=meshes/link_4.stl scale=0.001 0.001 0.001; visual mesh filename=meshes/link_4.stl scale=0.001 0.001 0.001
- added link link_5, mass 45.71412672440309; collision mesh filename=meshes/link_5.stl scale=0.001 0.001 0.001; visual mesh filename=meshes/link_5.stl scale=0.001 0.001 0.001
- added link link_6, mass 29.063646140411308; collision mesh filename=meshes/link_6.stl scale=0.001 0.001 0.001; visual mesh filename=meshes/link_6.stl scale=0.001 0.001 0.001
- added link tool0
Joints:
- removed joint j1
- removed joint j2
- removed joint j3
- removed joint j4
- removed joint j5
- removed joint j6
- added joint flange_to_tool0: type fixed, parent flange, child tool0, origin xyz=0 0 0 rpy=0 0 0
- added joint joint_1: type continuous, parent base_link, child link_1, origin xyz=0.0 0.0 0.342 rpy=0 0 0, axis 0.0 0.0 1.0
- added joint joint_2: type continuous, parent link_1, child link_2, origin xyz=0.69 -0.1535 0.188 rpy=0 0 0, axis 0.0 -1.0 0.0
- added joint joint_3: type continuous, parent link_2, child link_3, origin xyz=0.0 -0.1115 1.28 rpy=0 0 0, axis 0.0 1.0 0.0
- added joint joint_4: type continuous, parent link_3, child link_4, origin xyz=0.287 0.265 0.2 rpy=0 0 0, axis 1.0 0.0 0.0
- added joint joint_5: type continuous, parent link_4, child link_5, origin xyz=1.6355 0.095 0.0 rpy=0 0 0, axis -0.0 -1.0 -0.0
- added joint joint_6: type continuous, parent link_5, child link_6, origin xyz=0.165 -0.095 0.0 rpy=0 0 0, axis 1.0 0.0 0.0
- added joint link_6_to_flange: type fixed, parent link_6, child flange, origin xyz=0 0 0 rpy=0 1.57 0
- joint counter_cylinder: child IRB6750S_All_OC_00_CYL_CAD_v1_1 -> counter_cylinder; parent IRB6750S_All_OC_00_LINK01_CAD_v1_1 -> link_1
