Commit message: before messing with it

File: library/ABB/CRB15000_5kg_950_v1/CRB15000_5kg_950.urdf (robot description, URDF)
Before this commit: robot CRB15000_5kg_950, 9 links, 8 joints
Joints:
- joint joint_1: limit lower=3.14159 upper=-3.14159 effort=175.44 velocity=2.181 -> lower=-3.14159 upper=3.14159 effort=175.44 velocity=2.181
- joint joint_2: limit lower=3.14159 upper=-3.14159 effort=175.44 velocity=2.181 -> lower=-3.14159 upper=3.14159 effort=175.44 velocity=2.181
- joint joint_3: limit lower=-3.927 upper=1.483 effort=90.6 velocity=2.444 -> lower=-3.92699 upper=0.95993 effort=90.6 velocity=2.444
- joint joint_4: limit lower=3.14159 upper=-3.14159 effort=18.72 velocity=3.491 -> lower=-3.14159 upper=3.14159 effort=18.72 velocity=3.491
- joint joint_5: limit lower=3.14159 upper=-3.14159 effort=21.44 velocity=3.491 -> lower=-3.14159 upper=3.14159 effort=21.44 velocity=3.491
- joint joint_6: limit lower=-4.712 upper=4.712 effort=9.2 velocity=3.491 -> lower=-4.71239 upper=4.71239 effort=9.2 velocity=3.491

Commit message: good crb15000 5

File: library/ABB/CRB15000_5kg_950_v1/CRB15000_5kg_950.urdf (robot description, URDF)
Before this commit: robot CRB15000_5kg_950, 9 links, 8 joints
Joints:
- joint joint_1: axis 0.0 0.0 -1.0 -> 0.0 0.0 1.0; origin xyz=0.0 0.0 0.1885 rpy=0 0 0 -> xyz=0.0 0.0 0.265 rpy=0 0 0
- joint joint_2: axis 0.0 -1.0 0.0 -> 0.0 1.0 0.0; origin xyz=-0.0 -0.085 0.0765 rpy=0 0 0 -> xyz=-0.0 0.0 0.0 rpy=0 0 0
- joint joint_3: axis 0.0 -1.0 0.0 -> 0.0 1.0 0.0; origin xyz=0.0 -0.001 0.444 rpy=0 0 0 -> xyz=0.0 0.0 0.444 rpy=0 0 0
- joint joint_4: origin xyz=0.096 0.086 0.11 rpy=0 0 0 -> xyz=0.095 0.0 0.11 rpy=0 0 0
- joint joint_5: axis 0.0 -1.0 0.0 -> 0.0 1.0 0.0; origin xyz=0.374 0.0745 0.0 rpy=0 0 0 -> xyz=0.375 0.0 0.0 rpy=0 0 0
- joint joint_6: origin xyz=0.068 -0.0745 0.08 rpy=0 0 0 -> xyz=0.067 0.0 0.08 rpy=0 0 0

Commit message: fine tune CRB15000_5kg

File: library/ABB/CRB15000_5kg_950_v1/CRB15000_5kg_950.urdf (robot description, URDF)
Before this commit: robot CRB15000_5kg_950, 9 links, 8 joints
Joints:
- joint joint_4: origin xyz=0.095 0.0 0.11 rpy=0 0 0 -> xyz=0.0 0.0 0.11 rpy=0 0 0
- joint joint_5: origin xyz=0.375 0.0 0.0 rpy=0 0 0 -> xyz=0.47 0.0 0.0 rpy=0 0 0
- joint joint_6: origin xyz=0.067 0.0 0.08 rpy=0 0 0 -> xyz=0.101 0.0 0.08 rpy=0 0 0

Commit message: CRB15000_5kg refinement (#9)
Unit tests and tweaking to match manual specs

File: library/ABB/CRB15000_5kg_950_v1/CRB15000_5kg_950.urdf (robot description, URDF)
Before this commit: robot CRB15000_5kg_950, 9 links, 8 joints
Joints:
- joint joint_1: axis 0.0 0.0 -1.0 -> 0.0 0.0 1.0; limit lower=3.14159 upper=-3.14159 effort=175.44 velocity=2.181 -> lower=-3.14159 upper=3.14159 effort=175.44 velocity=2.181; origin xyz=0.0 0.0 0.1885 rpy=0 0 0 -> xyz=0.0 0.0 0.265 rpy=0 0 0
- joint joint_2: axis 0.0 -1.0 0.0 -> 0.0 1.0 0.0; limit lower=3.14159 upper=-3.14159 effort=175.44 velocity=2.181 -> lower=-3.14159 upper=3.14159 effort=175.44 velocity=2.181; origin xyz=-0.0 -0.085 0.0765 rpy=0 0 0 -> xyz=-0.0 0.0 0.0 rpy=0 0 0
- joint joint_3: axis 0.0 -1.0 0.0 -> 0.0 1.0 0.0; limit lower=-3.927 upper=1.483 effort=90.6 velocity=2.444 -> lower=-3.92699 upper=0.95993 effort=90.6 velocity=2.444; origin xyz=0.0 -0.001 0.444 rpy=0 0 0 -> xyz=0.0 0.0 0.444 rpy=0 0 0
- joint joint_4: limit lower=3.14159 upper=-3.14159 effort=18.72 velocity=3.491 -> lower=-3.14159 upper=3.14159 effort=18.72 velocity=3.491; origin xyz=0.096 0.086 0.11 rpy=0 0 0 -> xyz=0.0 0.0 0.11 rpy=0 0 0
- joint joint_5: axis 0.0 -1.0 0.0 -> 0.0 1.0 0.0; limit lower=3.14159 upper=-3.14159 effort=21.44 velocity=3.491 -> lower=-3.14159 upper=3.14159 effort=21.44 velocity=3.491; origin xyz=0.374 0.0745 0.0 rpy=0 0 0 -> xyz=0.47 0.0 0.0 rpy=0 0 0
- joint joint_6: limit lower=-4.712 upper=4.712 effort=9.2 velocity=3.491 -> lower=-4.71239 upper=4.71239 effort=9.2 velocity=3.491; origin xyz=0.068 -0.0745 0.08 rpy=0 0 0 -> xyz=0.101 0.0 0.08 rpy=0 0 0
