Commit message: good

File: library/ABB/CRB15000_10kg_152_v1/CRB15000_10kg_152.urdf (robot description, URDF)
Before this commit: robot CRB15000_10kg_152, 9 links, 8 joints
Joints:
- joint joint_1: axis 0.0 0.0 -1.0 -> 0.0 0.0 1.0; origin xyz=0.0 0.0 0.215 rpy=0 0 0 -> xyz=0.0 0.0 0.218 rpy=0 0 0
- joint joint_2: origin xyz=0.15 -0.09615 0.185014 rpy=0 0 0 -> xyz=0.15 0.0 0.182 rpy=0 0 0
- joint joint_3: axis 0.0 -1.0 0.0 -> 0.0 1.0 0.0; origin xyz=0.0 0.01115 0.706986 rpy=0 0 0 -> xyz=0.0 0.0 0.707 rpy=0 0 0
- joint joint_4: origin xyz=0.096 0.085 0.11 rpy=0 0 0 -> xyz=0.0 0.0 0.110 rpy=0 0 0
- joint joint_5: axis 0.0 -1.0 0.0 -> 0.0 1.0 0.0; origin xyz=0.540883 0.0755 0.0 rpy=0 0 0 -> xyz=0.637 0.0 0.0 rpy=0 0 0
- joint joint_6: origin xyz=0.068117 -0.0755 0.08 rpy=0 0 0 -> xyz=0.101 0.0 0.080 rpy=0 0 0
