Commit message: checkpoint

File: library/ABB/CRB15000_12kg_127_v1/CRB15000_12kg_127.urdf (robot description, URDF)
Before this commit: robot CRB15000_12_127, 9 links, 8 joints
Joints:
- joint joint_1: axis -0.0 0.0 1.0 -> 0.0 0.0 1.0
- joint joint_2: axis 0.0 -1.0 -0.0 -> 0.0 1.0 0.0
- joint joint_3: axis 0.0 -1.0 -0.0 -> 0.0 1.0 -0.0
- joint joint_4: axis -1.0 0.0 -0.0 -> 1.0 0.0 -0.0
- joint joint_5: axis 0.0 -1.0 0.0 -> 0.0 1.0 0.0
- joint joint_6: axis -1.0 0.0 -0.0 -> 1.0 0.0 -0.0

Commit message: crb12 joints correct

File: library/ABB/CRB15000_12kg_127_v1/CRB15000_12kg_127.urdf (robot description, URDF)
Before this commit: robot CRB15000_12_127, 9 links, 8 joints
Joints:
- joint joint_1: origin xyz=0.0 0.0 0.181677 rpy=0 0 0 -> xyz=0.0 0.0 0.0 rpy=0 0 0
- joint joint_2: origin xyz=0.0 -0.09615 0.156323 rpy=0 0 0 -> xyz=0.0 0.0 0.338 rpy=0 0 0
- joint joint_3: axis 0.0 1.0 -0.0 -> 0.0 1.0 0.0; origin xyz=0.0 0.00985 0.707 rpy=0 0 0 -> xyz=0.0 0.0 0.707 rpy=0 0 0
- joint joint_4: axis 1.0 0.0 -0.0 -> 0.0 0.0 1.0; origin xyz=0.097 0.0863 0.11 rpy=0 0 0 -> xyz=0.0 0.0 0.110 rpy=0 0 0
- joint joint_5: origin xyz=0.437 0.0745 0.0 rpy=0 0 0 -> xyz=0.534 0.0 0.00 rpy=0 0 0
- joint joint_6: axis 1.0 0.0 -0.0 -> 0.0 0.0 1.0; origin xyz=0.0685 -0.0745 0.08 rpy=0 0 0 -> xyz=0.101 0.0 0.080 rpy=0 0 0
- joint joint_flange: origin xyz=0 0 0 rpy=0 1.57 0 -> xyz=0 0 0 rpy=0 0 0

Commit message: CRB15000 12kg fine tuning (#12)

File: library/ABB/CRB15000_12kg_127_v1/CRB15000_12kg_127.urdf (robot description, URDF)
Before this commit: robot CRB15000_12_127, 9 links, 8 joints
Joints:
- joint joint_1: axis -0.0 0.0 1.0 -> 0.0 0.0 1.0; origin xyz=0.0 0.0 0.181677 rpy=0 0 0 -> xyz=0.0 0.0 0.0 rpy=0 0 0
- joint joint_2: axis 0.0 -1.0 -0.0 -> 0.0 1.0 0.0; origin xyz=0.0 -0.09615 0.156323 rpy=0 0 0 -> xyz=0.0 0.0 0.338 rpy=0 0 0
- joint joint_3: axis 0.0 -1.0 -0.0 -> 0.0 1.0 0.0; origin xyz=0.0 0.00985 0.707 rpy=0 0 0 -> xyz=0.0 0.0 0.707 rpy=0 0 0
- joint joint_4: axis -1.0 0.0 -0.0 -> 0.0 0.0 1.0; origin xyz=0.097 0.0863 0.11 rpy=0 0 0 -> xyz=0.0 0.0 0.110 rpy=0 0 0
- joint joint_5: axis 0.0 -1.0 0.0 -> 0.0 1.0 0.0; origin xyz=0.437 0.0745 0.0 rpy=0 0 0 -> xyz=0.534 0.0 0.00 rpy=0 0 0
- joint joint_6: axis -1.0 0.0 -0.0 -> 0.0 0.0 1.0; origin xyz=0.0685 -0.0745 0.08 rpy=0 0 0 -> xyz=0.101 0.0 0.080 rpy=0 0 0
- joint joint_flange: origin xyz=0 0 0 rpy=0 1.57 0 -> xyz=0 0 0 rpy=0 0 0

Commit message: 12kg fix

File: library/ABB/CRB15000_12kg_127_v1/CRB15000_12kg_127.urdf (robot description, URDF)
Before this commit: robot CRB15000_12_127, 9 links, 8 joints
Links:
- link base_link: mass 43.32183419472872 -> 5
- link flange: mass 0.1 -> 5
- link link_1: mass 41.02562588128756 -> 5
- link link_2: mass 70.93334832681374 -> 5
- link link_3: mass 26.381731962312585 -> 5
- link link_4: mass 27.702812566356673 -> 5
- link link_5: mass 23.63754989165508 -> 5
- link link_6: mass 1.1500367505463056 -> 5
- link tool0: mass 0.01 -> 5
Joints:
- joint joint_4: axis 0.0 0.0 1.0 -> 1.0 0.0 0.0
- joint joint_6: axis 0.0 0.0 1.0 -> 1.0 0.0 0.0
- joint joint_flange: origin xyz=0 0 0 rpy=0 0 0 -> xyz=0 0 0 rpy=0 1.57 0
