Commit message: work on 1100

File: library/ABB/IRB1100_4kg_475_STD_v1/IRB1100_4kg_475_STD.urdf (robot description, URDF)
Before this commit: robot IRB1100_4kg_475_STD, 9 links, 8 joints
Joints:
- joint joint_2: axis 0.0 -1.0 0.0 -> 0.0 1.0 0.0; origin xyz=0.0 -0.0525 0.181 rpy=0 0 0 -> xyz=0.0 0.0 0.181 rpy=0 0 0
- joint joint_3: axis 0.0 -1.0 0.0 -> 0.0 1.0 0.0; origin xyz=0.0 -0.0105 0.225 rpy=0 0 0 -> xyz=0.0 0.0 0.210 rpy=0 0 0
- joint joint_4: origin xyz=0.0725 0.063 0.01 rpy=0 0 0 -> xyz=0.0 0.0 0.025 rpy=0 0 0
- joint joint_5: axis 0.0 -1.0 0.0 -> 0.0 1.0 0.0; origin xyz=0.1775 0.0265 0.0 rpy=0 0 0 -> xyz=0.314 0.0 0.0 rpy=0 0 0
- joint joint_6: axis -1.0 0.0 0.0 -> 1.0 0.0 0.0; origin xyz=0.056 -0.0265 0.0 rpy=0 0 0 -> xyz=0.0 0.0 0.0 rpy=0 0 0
