Commit message: IRB1200_5_90_STD joints good

File: library/ABB/IRB1200_5_90_STD_v1/IRB1200_5_90_STD.urdf (robot description, URDF)
Before this commit: robot IRB1200_5_90_STD, 9 links, 8 joints
Joints:
- joint joint_1: origin xyz=0.0 0.0 0.219 rpy=0 0 0 -> xyz=0.0 0.0 0.0 rpy=0 0 0
- joint joint_2: origin xyz=0.0 -0.0605 0.1801 rpy=0 0 0 -> xyz=0.0 0.0 0.399 rpy=0 0 0
- joint joint_3: axis 0.0 -1.0 0.0 -> 0.0 1.0 0.0; origin xyz=0.0 0.0025 0.448 rpy=0 0 0 -> xyz=0.0 0.0 0.448 rpy=0 0 0
- joint joint_4: axis -1.0 0.0 0.0 -> 1.0 0.0 0.0; origin xyz=0.2885 0.058 0.042 rpy=0 0 0 -> xyz=0.451 0.0 0.042 rpy=0 0 0
- joint joint_5: origin xyz=0.1625 -0.0285 0.0 rpy=0 0 0 -> xyz=0.0 0.0 0.0 rpy=0 0 0
- joint joint_6: origin xyz=0.077 0.0285 0.0 rpy=0 0 0 -> xyz=0.082 0.0 0.0 rpy=0 0 0

Commit message: regen usd

File: library/ABB/IRB1200_5_90_STD_v1/IRB1200_5_90_STD.urdf (robot description, URDF)
Before this commit: robot IRB1200_5_90_STD, 9 links, 8 joints
Links:
- link base_link: mass 83.56354769083484 -> 9
- link link_1: mass 47.59365241562889 -> 7
- link link_2: mass 0.0002346193667311735 -> 4.5
- link link_3: mass 50.4799691302992 -> 3.5
- link link_4: mass 13.07948314741883 -> 2.5
- link link_5: mass 4.044605310431727 -> 1.5
- link link_6: mass 0.03376885335108457 -> 0.75

Commit message: IRB1200_5_90_STD refined (#15)

File: library/ABB/IRB1200_5_90_STD_v1/IRB1200_5_90_STD.urdf (robot description, URDF)
Before this commit: robot IRB1200_5_90_STD, 9 links, 8 joints
Links:
- link base_link: mass 83.56354769083484 -> 9
- link link_1: mass 47.59365241562889 -> 7
- link link_2: mass 0.0002346193667311735 -> 4.5
- link link_3: mass 50.4799691302992 -> 3.5
- link link_4: mass 13.07948314741883 -> 2.5
- link link_5: mass 4.044605310431727 -> 1.5
- link link_6: mass 0.03376885335108457 -> 0.75
Joints:
- joint joint_1: origin xyz=0.0 0.0 0.219 rpy=0 0 0 -> xyz=0.0 0.0 0.0 rpy=0 0 0
- joint joint_2: origin xyz=0.0 -0.0605 0.1801 rpy=0 0 0 -> xyz=0.0 0.0 0.399 rpy=0 0 0
- joint joint_3: axis 0.0 -1.0 0.0 -> 0.0 1.0 0.0; origin xyz=0.0 0.0025 0.448 rpy=0 0 0 -> xyz=0.0 0.0 0.448 rpy=0 0 0
- joint joint_4: axis -1.0 0.0 0.0 -> 1.0 0.0 0.0; origin xyz=0.2885 0.058 0.042 rpy=0 0 0 -> xyz=0.451 0.0 0.042 rpy=0 0 0
- joint joint_5: origin xyz=0.1625 -0.0285 0.0 rpy=0 0 0 -> xyz=0.0 0.0 0.0 rpy=0 0 0
- joint joint_6: origin xyz=0.077 0.0285 0.0 rpy=0 0 0 -> xyz=0.082 0.0 0.0 rpy=0 0 0
