Commit message: fix urdf and USD

File: library/ABB/IRB1200H_5_90_STD_v1/IRB1200H_5_90_STD.urdf (robot description, URDF)
Before this commit: robot IRB1200H_5_90_STD, 9 links, 8 joints
Links:
- link base_link: mass 83.56281675930393 -> 9
- link link_1: mass 47.66891611618349 -> 7
- link link_2: mass 62.596941650298746 -> 4.5
- link link_3: mass 50.251919251788294 -> 3.5
- link link_4: mass 14.103086555281287 -> 2.5
- link link_5: mass 4.542326712154526 -> 1.5
- link link_6: mass 0.03668180966446797 -> 0.75
Joints:
- joint joint_1: axis 0.0 0.0 -1.0 -> 0.0 0.0 1.0; origin xyz=0.0 0.0 0.219 rpy=0 0 0 -> xyz=0.0 0.0 0.0 rpy=0 0 0
- joint joint_2: axis 0.0 -1.0 0.0 -> 0.0 1.0 0.0; origin xyz=0.0 0.06 0.1801 rpy=0 0 0 -> xyz=0.0 0.0 0.399 rpy=0 0 0
- joint joint_3: axis 0.0 -1.0 0.0 -> 0.0 1.0 0.0; origin xyz=0.0 0.004 0.448 rpy=0 0 0 -> xyz=0.0 0.0 0.448 rpy=0 0 0
- joint joint_4: origin xyz=0.2885 -0.064 0.041489 rpy=0 0 0 -> xyz=0.451 0.0 0.042 rpy=0 0 0
- joint joint_5: axis 0.0 -1.0 0.0 -> 0.0 1.0 0.0; origin xyz=0.162491 0.0255 0.000511 rpy=0 0 0 -> xyz=0.0 0.0 0.0 rpy=0 0 0
- joint joint_6: origin xyz=0.085509 -0.025514 1.2e-05 rpy=0 0 0 -> xyz=0.082 0.0 0.0 rpy=0 0 0
