Commit message: RS Models and Thumbnails

File: library/Kawasaki/RS003N_A001_v2/RS003N_A001.urdf (robot description, URDF)
Before this commit: robot RS003N_A001, 7 links, 6 joints
Links:
- removed link RS003N_A001_J1_1
- removed link RS003N_A001_J2_1
- removed link RS003N_A001_J3_1
- removed link RS003N_A001_J4_1
- removed link RS003N_A001_J5_1
- removed link RS003N_A001_J6_1
- added link flange, mass 0.1
- added link link_1, mass 23.918879150979507; collision mesh filename=meshes/link_1.stl scale=0.001 0.001 0.001; visual mesh filename=meshes/link_1.stl scale=0.001 0.001 0.001
- added link link_2, mass 35.91526155004196; collision mesh filename=meshes/link_2.stl scale=0.001 0.001 0.001; visual mesh filename=meshes/link_2.stl scale=0.001 0.001 0.001
- added link link_3, mass 26.756330259119952; collision mesh filename=meshes/link_3.stl scale=0.001 0.001 0.001; visual mesh filename=meshes/link_3.stl scale=0.001 0.001 0.001
- added link link_4, mass 5.667470646724205; collision mesh filename=meshes/link_4.stl scale=0.001 0.001 0.001; visual mesh filename=meshes/link_4.stl scale=0.001 0.001 0.001
- added link link_5, mass 2.424679107191323; collision mesh filename=meshes/link_5.stl scale=0.001 0.001 0.001; visual mesh filename=meshes/link_5.stl scale=0.001 0.001 0.001
- added link link_6, mass 0.08152820359979351; collision mesh filename=meshes/link_6.stl scale=0.001 0.001 0.001; visual mesh filename=meshes/link_6.stl scale=0.001 0.001 0.001
- added link tool0, mass 0.01
Joints:
- removed joint j1
- removed joint j2
- removed joint j3
- removed joint j4
- removed joint j5
- removed joint j6
- added joint joint_1: type revolute, parent base_link, child link_1, origin xyz=0.001209 -0.001085 0.166 rpy=0 0 0, axis 0.0 0.0 1.0, limit lower=-3.14159 upper=3.14159 effort=100.0 velocity=3.0
- added joint joint_2: type revolute, parent link_1, child link_2, origin xyz=-0.070209 0.121085 0.084 rpy=0 0 0, axis 1.0 0.0 0.0, limit lower=-1.74533 upper=2.26893 effort=100.0 velocity=3.0
- added joint joint_3: type revolute, parent link_2, child link_3, origin xyz=0.006458 0.0 0.25 rpy=0 0 0, axis 1.0 0.0 0.0, limit lower=-3.49066 upper=1.22173 effort=100.0 velocity=3.0
- added joint joint_4: type revolute, parent link_3, child link_4, origin xyz=0.062542 0.0 0.1435 rpy=0 0 0, axis 0.0 0.0 1.0, limit lower=-3.14159 upper=3.14159 effort=50.0 velocity=6.0
- added joint joint_5: type revolute, parent link_4, child link_5, origin xyz=-0.026458 0.0 0.1065 rpy=0 0 0, axis 1.0 0.0 0.0, limit lower=-2.26893 upper=2.26893 effort=50.0 velocity=6.0
- added joint joint_6: type revolute, parent link_5, child link_6, origin xyz=0.026458 0.0 0.0715 rpy=0 0 0, axis 0.0 0.0 1.0, limit lower=-4.71239 upper=4.71239 effort=50.0 velocity=10.0
- added joint joint_flange: type fixed, parent link_6, child flange, origin xyz=0 0.12 0 rpy=0 1.57 0
- added joint joint_tool0: type fixed, parent flange, child tool0, origin xyz=0 0 0 rpy=0 0 0

File: library/Kawasaki/RS005L_A001_v2/RS005L_A001.urdf (robot description, URDF)
Before this commit: robot RS005L_A001, 7 links, 6 joints
Links:
- removed link RS005L_A001_J1_1
- removed link RS005L_A001_J2_1
- removed link RS005L_A001_J3_1
- removed link RS005L_A001_J4_1
- removed link RS005L_A001_J5_1
- removed link RS005L_A001_J6_1
- added link flange, mass 0.1
- added link link_1, mass 43.016701704037; collision mesh filename=meshes/link_1.stl scale=0.001 0.001 0.001; visual mesh filename=meshes/link_1.stl scale=0.001 0.001 0.001
- added link link_2, mass 56.20157888391649; collision mesh filename=meshes/link_2.stl scale=0.001 0.001 0.001; visual mesh filename=meshes/link_2.stl scale=0.001 0.001 0.001
- added link link_3, mass 42.88417286163072; collision mesh filename=meshes/link_3.stl scale=0.001 0.001 0.001; visual mesh filename=meshes/link_3.stl scale=0.001 0.001 0.001
- added link link_4, mass 12.927091362464212; collision mesh filename=meshes/link_4.stl scale=0.001 0.001 0.001; visual mesh filename=meshes/link_4.stl scale=0.001 0.001 0.001
- added link link_5, mass 2.72160915616873; collision mesh filename=meshes/link_5.stl scale=0.001 0.001 0.001; visual mesh filename=meshes/link_5.stl scale=0.001 0.001 0.001
- added link link_6, mass 0.09497074251738848; collision mesh filename=meshes/link_6.stl scale=0.001 0.001 0.001; visual mesh filename=meshes/link_6.stl scale=0.001 0.001 0.001
- added link tool0, mass 0.01
Joints:
- removed joint Revolute_1
- removed joint Revolute_2
- removed joint Revolute_3
- removed joint Revolute_4
- removed joint Revolute_5
- removed joint Revolute_6
- added joint joint_1: type revolute, parent base_link, child link_1, origin xyz=0.0 7e-06 0.165 rpy=0 0 0, axis 0.0 0.0 1.0, limit lower=-3.14159 upper=3.14159 effort=100 velocity=3.14
- added joint joint_2: type revolute, parent link_1, child link_2, origin xyz=-0.0585 0.104993 0.13 rpy=0 0 0, axis 1.0 0.0 0.0, limit lower=-2.26893 upper=2.26893 effort=100 velocity=3.14
- added joint joint_3: type revolute, parent link_2, child link_3, origin xyz=-0.0205 0.0 0.38 rpy=0 0 0, axis -1.0 0.0 -0.0, limit lower=-3.49066 upper=1.22173 effort=100 velocity=3.14
- added joint joint_4: type revolute, parent link_3, child link_4, origin xyz=0.078978 -0.08 0.15 rpy=0 0 0, axis 0.0 0.0 1.0, limit lower=-3.14159 upper=3.14159 effort=50 velocity=6.28
- added joint joint_5: type revolute, parent link_4, child link_5, origin xyz=-0.029478 0.0 0.26 rpy=0 0 0, axis 1.0 0.0 0.0, limit lower=-2.26893 upper=2.26893 effort=50 velocity=6.28
- added joint joint_6: type revolute, parent link_5, child link_6, origin xyz=0.0295 0.0 0.072 rpy=0 0 0, axis -0.0 -0.0 1.0, limit lower=-3.14159 upper=3.14159 effort=50 velocity=6.28
- added joint joint_flange: type fixed, parent link_6, child flange, origin xyz=0 0 0 rpy=0 1.57 0
- added joint joint_tool0: type fixed, parent flange, child tool0, origin xyz=0 0 0 rpy=0 0 0

File: library/Kawasaki/RS005N_A001_v2/RS005N_A001.urdf (robot description, URDF)
Before this commit: robot RS005N_A001, 7 links, 6 joints
Links:
- removed link RS005N_A001_J1_1
- removed link RS005N_A001_J2_1
- removed link RS005N_A001_J3_1
- removed link RS005N_A001_J4_1
- removed link RS005N_A001_J5_1
- removed link RS005N_A001_J6_1
- added link flange, mass 0.1
- added link link_1, mass 43.016701704037; collision mesh filename=meshes/link_1.stl scale=0.001 0.001 0.001; visual mesh filename=meshes/link_1.stl scale=0.001 0.001 0.001
- added link link_2, mass 39.75189074475072; collision mesh filename=meshes/link_2.stl scale=0.001 0.001 0.001; visual mesh filename=meshes/link_2.stl scale=0.001 0.001 0.001
- added link link_3, mass 42.49231008796781; collision mesh filename=meshes/link_3.stl scale=0.001 0.001 0.001; visual mesh filename=meshes/link_3.stl scale=0.001 0.001 0.001
- added link link_4, mass 8.018755692417622; collision mesh filename=meshes/link_4.stl scale=0.001 0.001 0.001; visual mesh filename=meshes/link_4.stl scale=0.001 0.001 0.001
- added link link_5, mass 2.7318577890089277; collision mesh filename=meshes/link_5.stl scale=0.001 0.001 0.001; visual mesh filename=meshes/link_5.stl scale=0.001 0.001 0.001
- added link link_6, mass 0.11374170714458348; collision mesh filename=meshes/link_6.stl scale=0.001 0.001 0.001; visual mesh filename=meshes/link_6.stl scale=0.001 0.001 0.001
- added link tool0, mass 0.01
Joints:
- removed joint j1
- removed joint j2
- removed joint j3
- removed joint j4
- removed joint j5
- removed joint j6
- added joint joint_1: type revolute, parent base_link, child link_1, origin xyz=0.0 7e-06 0.165 rpy=0 0 0, axis 0.0 0.0 1.0, limit lower=-3.14159 upper=3.14159 effort=147.0 velocity=3.84
- added joint joint_2: type revolute, parent link_1, child link_2, origin xyz=-0.0585 0.104993 0.13 rpy=0 0 0, axis 1.0 0.0 0.0, limit lower=-1.5708 upper=2.3562 effort=147.0 velocity=3.32
- added joint joint_3: type revolute, parent link_2, child link_3, origin xyz=-0.0205 0.0 0.28 rpy=0 0 0, axis 1.0 0.0 0.0, limit lower=-2.8798 upper=2.8798 effort=147.0 velocity=3.84
- added joint joint_4: type revolute, parent link_3, child link_4, origin xyz=0.078978 -0.08 0.15 rpy=0 0 0, axis 0.0 0.0 1.0, limit lower=-3.14159 upper=3.14159 effort=29.4 velocity=6.98
- added joint joint_5: type revolute, parent link_4, child link_5, origin xyz=-0.029478 0.0 0.16 rpy=0 0 0, axis 1.0 0.0 0.0, limit lower=-2.0944 upper=2.0944 effort=29.4 velocity=6.98
- added joint joint_6: type revolute, parent link_5, child link_6, origin xyz=0.0295 0.0 0.0655 rpy=0 0 0, axis 0.0 0.0 1.0, limit lower=-6.28319 upper=6.28319 effort=9.8 velocity=10.5
- added joint joint_flange: type fixed, parent link_6, child flange, origin xyz=0 0 0 rpy=0 1.57 0
- added joint joint_tool0: type fixed, parent flange, child tool0, origin xyz=0 0 0 rpy=0 0 0

File: library/Kawasaki/RS006L_A001_v2/RS006L_A001.urdf (robot description, URDF)
Before this commit: robot RS006L_A001, 7 links, 6 joints
Links:
- removed link RS006L_A001_J1_1
- removed link RS006L_A001_J2_1
- removed link RS006L_A001_J3_1
- removed link RS006L_A001_J4_1
- removed link RS006L_A001_J5_1
- removed link RS006L_A001_J6_1
- added link flange, mass 0.1
- added link link_1, mass 128.62439423296775; collision mesh filename=meshes/link_1.stl scale=0.001 0.001 0.001; visual mesh filename=meshes/link_1.stl scale=0.001 0.001 0.001
- added link link_2, mass 103.82770562805145; collision mesh filename=meshes/link_2.stl scale=0.001 0.001 0.001; visual mesh filename=meshes/link_2.stl scale=0.001 0.001 0.001
- added link link_3, mass 75.88480135521745; collision mesh filename=meshes/link_3.stl scale=0.001 0.001 0.001; visual mesh filename=meshes/link_3.stl scale=0.001 0.001 0.001
- added link link_4, mass 52.79047116312823; collision mesh filename=meshes/link_4.stl scale=0.001 0.001 0.001; visual mesh filename=meshes/link_4.stl scale=0.001 0.001 0.001
- added link link_5, mass 4.056209614474094; collision mesh filename=meshes/link_5.stl scale=0.001 0.001 0.001; visual mesh filename=meshes/link_5.stl scale=0.001 0.001 0.001
- added link link_6, mass 0.38905629501068684; collision mesh filename=meshes/link_6.stl scale=0.001 0.001 0.001; visual mesh filename=meshes/link_6.stl scale=0.001 0.001 0.001
- added link tool0, mass 0.01
Joints:
- removed joint Revolute_1
- removed joint Revolute_2
- removed joint Revolute_3
- removed joint Revolute_4
- removed joint Revolute_5
- removed joint Revolute_6
- added joint joint_1: type revolute, parent base_link, child link_1, origin xyz=0.0 0.0 0.184 rpy=0 0 0, axis 0.0 0.0 1.0, limit lower=-3.14159 upper=3.14159 effort=150.0 velocity=3.14
- added joint joint_2: type revolute, parent link_1, child link_2, origin xyz=0.15 0.1 0.246 rpy=0 0 0, axis -1.0 0.0 0.0, limit lower=-2.26893 upper=2.26893 effort=150.0 velocity=3.14
- added joint joint_3: type revolute, parent link_2, child link_3, origin xyz=-0.08 0.0 0.65 rpy=0 0 0, axis -1.0 0.0 0.0, limit lower=-3.49066 upper=1.22173 effort=150.0 velocity=3.14
- added joint joint_4: type revolute, parent link_3, child link_4, origin xyz=-0.07 0.0 0.1879 rpy=0 0 0, axis 0.0 0.0 1.0, limit lower=-3.14159 upper=3.14159 effort=60.0 velocity=6.28
- added joint joint_5: type revolute, parent link_4, child link_5, origin xyz=-0.031 0.0 0.7121 rpy=0 0 0, axis 1.0 0.0 0.0, limit lower=-2.26893 upper=2.26893 effort=60.0 velocity=6.28
- added joint joint_6: type revolute, parent link_5, child link_6, origin xyz=0.031 0.0 0.0665 rpy=0 0 0, axis -0.0 0.0 -1.0, limit lower=-3.14159 upper=3.14159 effort=60.0 velocity=6.28
- added joint joint_flange: type fixed, parent link_6, child flange, origin xyz=0 0 0 rpy=0 1.57 0
- added joint joint_tool0: type fixed, parent flange, child tool0, origin xyz=0 0 0 rpy=0 0 0

File: library/Kawasaki/RS007L_BC01_v1/RS007L_BC01.urdf (robot description, URDF)
Before this commit: robot RS007L_BC01, 7 links, 6 joints
Links:
- removed link RS007L_BC01_J1_1
- removed link RS007L_BC01_J2_1
- removed link RS007L_BC01_J3_1
- removed link RS007L_BC01_J4_1
- removed link RS007L_BC01_J5_1
- removed link RS007L_BC01_J6_1
- added link flange, mass 0.1
- added link link_1, mass 38.10131290624578; collision mesh filename=meshes/link_1.stl scale=0.001 0.001 0.001; visual mesh filename=meshes/link_1.stl scale=0.001 0.001 0.001
- added link link_2, mass 38.840353056430764; collision mesh filename=meshes/link_2.stl scale=0.001 0.001 0.001; visual mesh filename=meshes/link_2.stl scale=0.001 0.001 0.001
- added link link_3, mass 32.69573133878474; collision mesh filename=meshes/link_3.stl scale=0.001 0.001 0.001; visual mesh filename=meshes/link_3.stl scale=0.001 0.001 0.001
- added link link_4, mass 27.022539947933783; collision mesh filename=meshes/link_4.stl scale=0.001 0.001 0.001; visual mesh filename=meshes/link_4.stl scale=0.001 0.001 0.001
- added link link_5, mass 4.129208800242346; collision mesh filename=meshes/link_5.stl scale=0.001 0.001 0.001; visual mesh filename=meshes/link_5.stl scale=0.001 0.001 0.001
- added link link_6, mass 0.10554842236060766; collision mesh filename=meshes/link_6.stl scale=0.001 0.001 0.001; visual mesh filename=meshes/link_6.stl scale=0.001 0.001 0.001
- added link tool0, mass 0.01
Joints:
- removed joint Revolute_1
- removed joint Revolute_2
- removed joint Revolute_3
- removed joint Revolute_4
- removed joint Revolute_5
- removed joint Revolute_6
- added joint joint_1: type revolute, parent base_link, child link_1, origin xyz=0.0 0.0 0.187 rpy=0 0 0, axis 0.0 0.0 1.0, limit lower=-3.14159 upper=3.14159 effort=420.0 velocity=3.491
- added joint joint_2: type revolute, parent link_1, child link_2, origin xyz=0.055 0.0 0.173 rpy=0 0 0, axis 1.0 0.0 0.0, limit lower=-2.0944 upper=2.0944 effort=490.0 velocity=3.491
- added joint joint_3: type revolute, parent link_2, child link_3, origin xyz=0.02 0.0 0.455 rpy=0 0 0, axis 1.0 -0.0 0.0, limit lower=-3.14159 upper=3.14159 effort=194.0 velocity=3.491
- added joint joint_4: type revolute, parent link_3, child link_4, origin xyz=-0.075103 -0.0 0.108 rpy=0 0 0, axis -0.0 -0.0 1.0, limit lower=-3.14159 upper=3.14159 effort=49.0 velocity=6.283
- added joint joint_5: type revolute, parent link_4, child link_5, origin xyz=-0.026897 0.0 0.367 rpy=0 0 0, axis 1.0 -0.0 0.0, limit lower=-2.0944 upper=2.0944 effort=49.0 velocity=6.283
- added joint joint_6: type revolute, parent link_5, child link_6, origin xyz=0.027 0.0 0.06455 rpy=0 0 0, axis -0.0 0.0 1.0, limit lower=-4.71239 upper=4.71239 effort=20.0 velocity=6.283
- added joint joint_flange: type fixed, parent link_6, child flange, origin xyz=0 0 0 rpy=0 1.57 0
- added joint joint_tool0: type fixed, parent flange, child tool0, origin xyz=0 0 0 rpy=0 0 0

File: library/Kawasaki/RS007N_BC01_v1/RS007N_BC01.urdf (robot description, URDF)
Before this commit: robot RS007N_BC01, 7 links, 6 joints
Links:
- removed link RS007N_BC01_J1_1
- removed link RS007N_BC01_J2_1
- removed link RS007N_BC01_J3_1
- removed link RS007N_BC01_J4_1
- removed link RS007N_BC01_J5_1
- removed link RS007N_BC01_J6_1
- added link flange, mass 0.1
- added link link_1, mass 38.10131290624578; collision mesh filename=meshes/link_1.stl scale=0.001 0.001 0.001; visual mesh filename=meshes/link_1.stl scale=0.001 0.001 0.001
- added link link_2, mass 33.40803626291563; collision mesh filename=meshes/link_2.stl scale=0.001 0.001 0.001; visual mesh filename=meshes/link_2.stl scale=0.001 0.001 0.001
- added link link_3, mass 32.69573133878474; collision mesh filename=meshes/link_3.stl scale=0.001 0.001 0.001; visual mesh filename=meshes/link_3.stl scale=0.001 0.001 0.001
- added link link_4, mass 20.86130924821223; collision mesh filename=meshes/link_4.stl scale=0.001 0.001 0.001; visual mesh filename=meshes/link_4.stl scale=0.001 0.001 0.001
- added link link_5, mass 4.129208800242346; collision mesh filename=meshes/link_5.stl scale=0.001 0.001 0.001; visual mesh filename=meshes/link_5.stl scale=0.001 0.001 0.001
- added link link_6, mass 0.10554842236060766; collision mesh filename=meshes/link_6.stl scale=0.001 0.001 0.001; visual mesh filename=meshes/link_6.stl scale=0.001 0.001 0.001
- added link tool0, mass 0.01
Joints:
- removed joint Revolute_1
- removed joint Revolute_2
- removed joint Revolute_3
- removed joint Revolute_4
- removed joint Revolute_5
- removed joint Revolute_6
- added joint joint_1: type revolute, parent base_link, child link_1, origin xyz=0.0 0.0 0.187 rpy=0 0 0, axis 0.0 0.0 1.0, limit lower=-3.14159 upper=3.14159 effort=300 velocity=3.14
- added joint joint_2: type revolute, parent link_1, child link_2, origin xyz=0.055 0.0 0.173 rpy=0 0 0, axis 1.0 0.0 0.0, limit lower=-2.35619 upper=2.35619 effort=300 velocity=3.14
- added joint joint_3: type revolute, parent link_2, child link_3, origin xyz=0.02 0.0 0.355 rpy=0 0 0, axis 1.0 -0.0 0.0, limit lower=-2.79253 upper=0.6981 effort=150 velocity=3.14
- added joint joint_4: type revolute, parent link_3, child link_4, origin xyz=-0.075103 -0.0 0.108 rpy=0 0 0, axis -0.0 -0.0 1.0, limit lower=-4.71239 upper=4.71239 effort=50 velocity=6.28
- added joint joint_5: type revolute, parent link_4, child link_5, origin xyz=-0.034797 0.0 0.267 rpy=0 0 0, axis 1.0 -0.0 0.0, limit lower=-2.18166 upper=2.18166 effort=50 velocity=6.28
- added joint joint_6: type revolute, parent link_5, child link_6, origin xyz=0.0349 0.0 0.06455 rpy=0 0 0, axis -0.0 0.0 1.0, limit lower=-6.28319 upper=6.28319 effort=25 velocity=6.28
- added joint joint_flange: type fixed, parent link_6, child flange, origin xyz=0 0 0 rpy=0 1.57 0
- added joint joint_tool0: type fixed, parent flange, child tool0, origin xyz=0 0 0 rpy=0 0 0

File: library/Kawasaki/RS013N_AC01_v1/RS013N_AC01.urdf (robot description, URDF)
Before this commit: robot RS013N_AC01, 7 links, 6 joints
Links:
- removed link RS013N_AC01_J1_1
- removed link RS013N_AC01_J2_1
- removed link RS013N_AC01_J3_1
- removed link RS013N_AC01_J4_1
- removed link RS013N_AC01_J5_1
- removed link RS013N_AC01_J6_1
- added link flange, mass 0.1
- added link link_1, mass 171.7477703614906; collision mesh filename=meshes/link_1.stl scale=0.001 0.001 0.001; visual mesh filename=meshes/link_1.stl scale=0.001 0.001 0.001
- added link link_2, mass 129.8221396805681; collision mesh filename=meshes/link_2.stl scale=0.001 0.001 0.001; visual mesh filename=meshes/link_2.stl scale=0.001 0.001 0.001
- added link link_3, mass 72.92951822722108; collision mesh filename=meshes/link_3.stl scale=0.001 0.001 0.001; visual mesh filename=meshes/link_3.stl scale=0.001 0.001 0.001
- added link link_4, mass 52.077389951662894; collision mesh filename=meshes/link_4.stl scale=0.001 0.001 0.001; visual mesh filename=meshes/link_4.stl scale=0.001 0.001 0.001
- added link link_5, mass 4.204702678186262; collision mesh filename=meshes/link_5.stl scale=0.001 0.001 0.001; visual mesh filename=meshes/link_5.stl scale=0.001 0.001 0.001
- added link link_6, mass 0.15136116479950507; collision mesh filename=meshes/link_6.stl scale=0.001 0.001 0.001; visual mesh filename=meshes/link_6.stl scale=0.001 0.001 0.001
- added link tool0, mass 0.01
Joints:
- removed joint Revolute_1
- removed joint Revolute_2
- removed joint Revolute_3
- removed joint Revolute_4
- removed joint Revolute_5
- removed joint Revolute_6
- added joint joint_1: type revolute, parent base_link, child link_1, origin xyz=0.0 0.0 0.235 rpy=0 0 0, axis 0.0 0.0 1.0, limit lower=-3.14159 upper=3.14159 effort=300 velocity=3.1416
- added joint joint_2: type revolute, parent link_1, child link_2, origin xyz=0.073 0.0 0.27 rpy=0 0 0, axis 1.0 0.0 0.0, limit lower=-3.14159 upper=3.14159 effort=300 velocity=3.1416
- added joint joint_3: type revolute, parent link_2, child link_3, origin xyz=0.037 -0.0 0.7 rpy=0 0 0, axis 1.0 0.0 0.0, limit lower=-3.14159 upper=3.14159 effort=300 velocity=3.1416
- added joint joint_4: type revolute, parent link_3, child link_4, origin xyz=-0.11 0.0 0.1334 rpy=0 0 0, axis 0.0 0.0 1.0, limit lower=-3.14159 upper=3.14159 effort=100 velocity=4.3633
- added joint joint_5: type revolute, parent link_4, child link_5, origin xyz=-0.0349 0.0 0.6266 rpy=0 0 0, axis 1.0 0.0 0.0, limit lower=-3.14159 upper=3.14159 effort=100 velocity=4.3633
- added joint joint_6: type revolute, parent link_5, child link_6, origin xyz=0.0349 0.0 0.067 rpy=0 0 0, axis 0.0 0.0 1.0, limit lower=-4.71239 upper=4.71239 effort=50 velocity=4.3633
- added joint joint_flange: type fixed, parent link_6, child flange, origin xyz=0 0 0 rpy=0 1.57 0
- added joint joint_tool0: type fixed, parent flange, child tool0, origin xyz=0 0 0 rpy=0 0 0
