Commit message: RS Models and Thumbnails

File: library/Kawasaki/RS015X_B001_v1/RS015X_B001.urdf (robot description, URDF)
Before this commit: robot RS015X_B001, 7 links, 6 joints
Links:
- removed link RS015X_B001_J1_1
- removed link RS015X_B001_J2_1
- removed link RS015X_B001_J3_1
- removed link RS015X_B001_J4_1
- removed link RS015X_B001_J5_1
- removed link RS015X_B001_J6_1
- added link flange, mass 0.1
- added link link_1, mass 461.12398981682077; collision mesh filename=meshes/link_1.stl scale=0.001 0.001 0.001; visual mesh filename=meshes/link_1.stl scale=0.001 0.001 0.001
- added link link_2, mass 412.89081962234826; collision mesh filename=meshes/link_2.stl scale=0.001 0.001 0.001; visual mesh filename=meshes/link_2.stl scale=0.001 0.001 0.001
- added link link_3, mass 238.9958582792771; collision mesh filename=meshes/link_3.stl scale=0.001 0.001 0.001; visual mesh filename=meshes/link_3.stl scale=0.001 0.001 0.001
- added link link_4, mass 175.8337733882442; collision mesh filename=meshes/link_4.stl scale=0.001 0.001 0.001; visual mesh filename=meshes/link_4.stl scale=0.001 0.001 0.001
- added link link_5, mass 6.633599900730962; collision mesh filename=meshes/link_5.stl scale=0.001 0.001 0.001; visual mesh filename=meshes/link_5.stl scale=0.001 0.001 0.001
- added link link_6, mass 0.39757123901471203; collision mesh filename=meshes/link_6.stl scale=0.001 0.001 0.001; visual mesh filename=meshes/link_6.stl scale=0.001 0.001 0.001
- added link tool0, mass 0.01
Joints:
- removed joint j1
- removed joint j2
- removed joint j3
- removed joint j4
- removed joint j5
- removed joint j6
- added joint joint_1: type revolute, parent base_link, child link_1, origin xyz=0.0 0.0 0.249 rpy=0 0 0, axis 0.0 0.0 1.0, limit lower=-3.14159 upper=3.14159 effort=500.0 velocity=6.0
- added joint joint_2: type revolute, parent link_1, child link_2, origin xyz=0.035 0.15 0.431 rpy=0 0 0, axis 1.0 0.0 0.0, limit lower=-3.14159 upper=3.14159 effort=500.0 velocity=6.0
- added joint joint_3: type revolute, parent link_2, child link_3, origin xyz=0.087 0.0 1.15 rpy=0 0 0, axis 1.0 0.0 0.0, limit lower=-3.14159 upper=3.14159 effort=500.0 velocity=6.0
- added joint joint_4: type revolute, parent link_3, child link_4, origin xyz=-0.122 0.0 0.27 rpy=0 0 0, axis 0.0 0.0 1.0, limit lower=-3.14159 upper=3.14159 effort=500.0 velocity=6.0
- added joint joint_5: type revolute, parent link_4, child link_5, origin xyz=-0.042 0.0 1.58 rpy=0 0 0, axis 1.0 0.0 0.0, limit lower=-3.14159 upper=3.14159 effort=500.0 velocity=6.0
- added joint joint_6: type revolute, parent link_5, child link_6, origin xyz=0.042001 0.0 0.081 rpy=0 0 0, axis 0.0 0.0 1.0, limit lower=-3.14159 upper=3.14159 effort=500.0 velocity=6.0
- added joint joint_flange: type fixed, parent link_6, child flange, origin xyz=0 0 0 rpy=0 1.57 0
- added joint joint_tool0: type fixed, parent flange, child tool0, origin xyz=0 0 0 rpy=0 0 0

File: library/Kawasaki/RS020N_A001_v1/RS020N_A001.urdf (robot description, URDF)
Before this commit: robot RS020N_A001, 7 links, 6 joints
Links:
- removed link RS020N_A001_J1_1
- removed link RS020N_A001_J2_1
- removed link RS020N_A001_J3_1
- removed link RS020N_A001_J4_1
- removed link RS020N_A001_J5_1
- removed link RS020N_A001_J6_1
- added link flange, mass 0.1
- added link link_1, mass 181.6362691193184; collision mesh filename=meshes/link_1.stl scale=0.001 0.001 0.001; visual mesh filename=meshes/link_1.stl scale=0.001 0.001 0.001
- added link link_2, mass 163.889002973526; collision mesh filename=meshes/link_2.stl scale=0.001 0.001 0.001; visual mesh filename=meshes/link_2.stl scale=0.001 0.001 0.001
- added link link_3, mass 112.0588844871384; collision mesh filename=meshes/link_3.stl scale=0.001 0.001 0.001; visual mesh filename=meshes/link_3.stl scale=0.001 0.001 0.001
- added link link_4, mass 57.2635730535197; collision mesh filename=meshes/link_4.stl scale=0.001 0.001 0.001; visual mesh filename=meshes/link_4.stl scale=0.001 0.001 0.001
- added link link_5, mass 6.746554747014125; collision mesh filename=meshes/link_5.stl scale=0.001 0.001 0.001; visual mesh filename=meshes/link_5.stl scale=0.001 0.001 0.001
- added link link_6, mass 0.3970304122124492; collision mesh filename=meshes/link_6.stl scale=0.001 0.001 0.001; visual mesh filename=meshes/link_6.stl scale=0.001 0.001 0.001
- added link tool0, mass 0.01
Joints:
- removed joint j1
- removed joint j2
- removed joint j3
- removed joint j4
- removed joint j5
- removed joint j6
- added joint joint_1: type continuous, parent base_link, child link_1, origin xyz=0.0 0.0 0.199 rpy=0 0 0, axis 0.0 0.0 1.0
- added joint joint_2: type continuous, parent link_1, child link_2, origin xyz=0.06 0.15 0.266 rpy=0 0 0, axis 1.0 0.0 0.0
- added joint joint_3: type continuous, parent link_2, child link_3, origin xyz=0.028 0.0 0.77 rpy=0 0 0, axis 1.0 0.0 0.0
- added joint joint_4: type continuous, parent link_3, child link_4, origin xyz=-0.088 0.0 0.197 rpy=0 0 0, axis 0.0 0.0 1.0
- added joint joint_5: type continuous, parent link_4, child link_5, origin xyz=-0.0415 0.0 0.608 rpy=0 0 0, axis 1.0 0.0 0.0
- added joint joint_6: type continuous, parent link_5, child link_6, origin xyz=0.042001 0.0 0.081 rpy=0 0 0, axis 0.0 0.0 1.0
- added joint joint_flange: type fixed, parent link_6, child flange, origin xyz=0 0 0 rpy=0 1.57 0
- added joint joint_tool0: type fixed, parent flange, child tool0, origin xyz=0 0 0 rpy=0 0 0

File: library/Kawasaki/RS025N_AC01_v1/RS025N_AC01.urdf (robot description, URDF)
Before this commit: robot RS025N_AC01, 7 links, 6 joints
Links:
- removed link RS025N_AC01_J1_1
- removed link RS025N_AC01_J2_1
- removed link RS025N_AC01_J3_1
- removed link RS025N_AC01_J4_1
- removed link RS025N_AC01_J5_1
- removed link RS025N_AC01_J6_1
- added link flange, mass 0.1
- added link link_1, mass 239.81672104338398; collision mesh filename=meshes/link_1.stl scale=0.001 0.001 0.001; visual mesh filename=meshes/link_1.stl scale=0.001 0.001 0.001
- added link link_2, mass 246.92577724341461; collision mesh filename=meshes/link_2.stl scale=0.001 0.001 0.001; visual mesh filename=meshes/link_2.stl scale=0.001 0.001 0.001
- added link link_3, mass 163.13380863446162; collision mesh filename=meshes/link_3.stl scale=0.001 0.001 0.001; visual mesh filename=meshes/link_3.stl scale=0.001 0.001 0.001
- added link link_4, mass 87.64633037093972; collision mesh filename=meshes/link_4.stl scale=0.001 0.001 0.001; visual mesh filename=meshes/link_4.stl scale=0.001 0.001 0.001
- added link link_5, mass 10.376581535909532; collision mesh filename=meshes/link_5.stl scale=0.001 0.001 0.001; visual mesh filename=meshes/link_5.stl scale=0.001 0.001 0.001
- added link link_6, mass 0.2861491774605701; collision mesh filename=meshes/link_6.stl scale=0.001 0.001 0.001; visual mesh filename=meshes/link_6.stl scale=0.001 0.001 0.001
- added link tool0, mass 0.01
Joints:
- removed joint j1
- removed joint j2
- removed joint j3
- removed joint j4
- removed joint j5
- removed joint j6
- added joint joint_1: type revolute, parent base_link, child link_1, origin xyz=0.0 0.0 0.29 rpy=0 0 0, axis 0.0 0.0 1.0, limit lower=-3.14159 upper=3.14159 effort=500 velocity=3.316
- added joint joint_2: type revolute, parent link_1, child link_2, origin xyz=0.093 0.0 0.29 rpy=0 0 0, axis 1.0 0.0 0.0, limit lower=-1.309 upper=1.5708 effort=500 velocity=2.96
- added joint joint_3: type revolute, parent link_2, child link_3, origin xyz=0.05 0.0 0.885 rpy=0 0 0, axis 1.0 0.0 0.0, limit lower=-2.356 upper=2.094 effort=300 velocity=3.316
- added joint joint_4: type revolute, parent link_3, child link_4, origin xyz=-0.143 0.0 0.179 rpy=0 0 0, axis 0.0 0.0 1.0, limit lower=-3.14159 upper=3.14159 effort=80 velocity=6.98
- added joint joint_5: type revolute, parent link_4, child link_5, origin xyz=-0.048 0.0 0.821 rpy=0 0 0, axis 1.0 0.0 0.0, limit lower=-2.356 upper=2.356 effort=40 velocity=6.98
- added joint joint_6: type revolute, parent link_5, child link_6, origin xyz=0.048 0.0 0.0835 rpy=0 0 0, axis 0.0 0.0 1.0, limit lower=-6.28319 upper=6.28319 effort=20 velocity=10.47
- added joint joint_flange: type fixed, parent link_6, child flange, origin xyz=0 0 0 rpy=0 1.57 0
- added joint joint_tool0: type fixed, parent flange, child tool0, origin xyz=0 0 0 rpy=0 0 0

File: library/Kawasaki/RS030N_B001_v1/RS030N_B001.urdf (robot description, URDF)
Before this commit: robot RS030N_B001, 7 links, 6 joints
Links:
- removed link RS030N_B001_J1_1
- removed link RS030N_B001_J2_1
- removed link RS030N_B001_J3_1
- removed link RS030N_B001_J4_1
- removed link RS030N_B001_J5_1
- removed link RS030N_B001_J6_1
- added link flange, mass 0.1
- added link link_1, mass 462.0578622187538; collision mesh filename=meshes/link_1.stl scale=0.001 0.001 0.001; visual mesh filename=meshes/link_1.stl scale=0.001 0.001 0.001
- added link link_2, mass 357.1979641343307; collision mesh filename=meshes/link_2.stl scale=0.001 0.001 0.001; visual mesh filename=meshes/link_2.stl scale=0.001 0.001 0.001
- added link link_3, mass 238.65048189451747; collision mesh filename=meshes/link_3.stl scale=0.001 0.001 0.001; visual mesh filename=meshes/link_3.stl scale=0.001 0.001 0.001
- added link link_4, mass 154.12861681817174; collision mesh filename=meshes/link_4.stl scale=0.001 0.001 0.001; visual mesh filename=meshes/link_4.stl scale=0.001 0.001 0.001
- added link link_5, mass 14.869315016615895; collision mesh filename=meshes/link_5.stl scale=0.001 0.001 0.001; visual mesh filename=meshes/link_5.stl scale=0.001 0.001 0.001
- added link link_6, mass 2.5308375704525687; collision mesh filename=meshes/link_6.stl scale=0.001 0.001 0.001; visual mesh filename=meshes/link_6.stl scale=0.001 0.001 0.001
- added link tool0, mass 0.01
Joints:
- removed joint j1
- removed joint j2
- removed joint j3
- removed joint j4
- removed joint j5
- removed joint j6
- added joint joint_1: type revolute, parent base_link, child link_1, origin xyz=0.0 0.0 0.249 rpy=0 0 0, axis 0.0 0.0 1.0, limit lower=-3.14159 upper=3.14159 effort=1000 velocity=3.14
- added joint joint_2: type revolute, parent link_1, child link_2, origin xyz=0.035 0.15 0.431 rpy=0 0 0, axis 1.0 0.0 0.0, limit lower=-1.396 upper=2.356 effort=1000 velocity=3.14
- added joint joint_3: type revolute, parent link_2, child link_3, origin xyz=0.087 0.0 0.87 rpy=0 0 0, axis 1.0 0.0 0.0, limit lower=-2.269 upper=2.618 effort=1000 velocity=3.14
- added joint joint_4: type revolute, parent link_3, child link_4, origin xyz=-0.122 0.0 0.27 rpy=0 0 0, axis 0.0 0.0 1.0, limit lower=-4.71239 upper=4.71239 effort=300 velocity=5.23
- added joint joint_5: type revolute, parent link_4, child link_5, origin xyz=-0.0595 0.0 0.81 rpy=0 0 0, axis 1.0 0.0 0.0, limit lower=-2.094 upper=2.094 effort=300 velocity=5.23
- added joint joint_6: type revolute, parent link_5, child link_6, origin xyz=0.0595 0.0 0.1265 rpy=0 0 0, axis 0.0 -0.0 1.0, limit lower=-6.28319 upper=6.28319 effort=200 velocity=6.98
- added joint joint_flange: type fixed, parent link_6, child flange, origin xyz=0 0 0 rpy=0 1.57 0
- added joint joint_tool0: type fixed, parent flange, child tool0, origin xyz=0 0 0 rpy=0 0 0

File: library/Kawasaki/RS050N_B001_v1/RS050N_B001.urdf (robot description, URDF)
Before this commit: robot RS050N_B001, 7 links, 6 joints
Links:
- removed link RS050N_B001_J1_1
- removed link RS050N_B001_J2_1
- removed link RS050N_B001_J3_1
- removed link RS050N_B001_J4_1
- removed link RS050N_B001_J5_1
- removed link RS050N_B001_J6_1
- added link flange, mass 0.1
- added link link_1, mass 462.1630132570103; collision mesh filename=meshes/link_1.stl scale=0.001 0.001 0.001; visual mesh filename=meshes/link_1.stl scale=0.001 0.001 0.001
- added link link_2, mass 357.1989200421478; collision mesh filename=meshes/link_2.stl scale=0.001 0.001 0.001; visual mesh filename=meshes/link_2.stl scale=0.001 0.001 0.001
- added link link_3, mass 238.7528174086134; collision mesh filename=meshes/link_3.stl scale=0.001 0.001 0.001; visual mesh filename=meshes/link_3.stl scale=0.001 0.001 0.001
- added link link_4, mass 154.1284973473204; collision mesh filename=meshes/link_4.stl scale=0.001 0.001 0.001; visual mesh filename=meshes/link_4.stl scale=0.001 0.001 0.001
- added link link_5, mass 14.869297796496278; collision mesh filename=meshes/link_5.stl scale=0.001 0.001 0.001; visual mesh filename=meshes/link_5.stl scale=0.001 0.001 0.001
- added link link_6, mass 2.5308375706093287; collision mesh filename=meshes/link_6.stl scale=0.001 0.001 0.001; visual mesh filename=meshes/link_6.stl scale=0.001 0.001 0.001
- added link tool0, mass 0.01
Joints:
- removed joint j1
- removed joint j2
- removed joint j3
- removed joint j4
- removed joint j5
- removed joint j6
- added joint joint_1: type revolute, parent base_link, child link_1, origin xyz=0.0 0.0 0.249 rpy=0 0 0, axis 0.0 0.0 1.0, limit lower=-3.14159 upper=3.14159 effort=1000 velocity=2.0
- added joint joint_2: type revolute, parent link_1, child link_2, origin xyz=0.035 0.15 0.431 rpy=0 0 0, axis 1.0 0.0 0.0, limit lower=-3.14159 upper=3.14159 effort=1000 velocity=2.0
- added joint joint_3: type revolute, parent link_2, child link_3, origin xyz=0.087 0.0 0.87 rpy=0 0 0, axis 1.0 0.0 0.0, limit lower=-3.14159 upper=3.14159 effort=1000 velocity=2.0
- added joint joint_4: type revolute, parent link_3, child link_4, origin xyz=-0.122 0.0 0.27 rpy=0 0 0, axis 0.0 0.0 1.0, limit lower=-3.14159 upper=3.14159 effort=1000 velocity=2.0
- added joint joint_5: type revolute, parent link_4, child link_5, origin xyz=-0.0595 0.0 0.81 rpy=0 0 0, axis 1.0 0.0 0.0, limit lower=-3.14159 upper=3.14159 effort=1000 velocity=2.0
- added joint joint_6: type revolute, parent link_5, child link_6, origin xyz=0.0595 0.0 0.1265 rpy=0 0 0, axis 0.0 0.0 1.0, limit lower=-3.14159 upper=3.14159 effort=1000 velocity=2.0
- added joint joint_flange: type fixed, parent link_6, child flange, origin xyz=0 0 0 rpy=0 1.57 0
- added joint joint_tool0: type fixed, parent flange, child tool0, origin xyz=0 0 0 rpy=0 0 0

File: library/Kawasaki/RS080N_B001_v1/RS080N_B001.urdf (robot description, URDF)
Before this commit: robot RS080N_B001, 7 links, 6 joints
Links:
- removed link RS080N_B001_J1_1
- removed link RS080N_B001_J2_1
- removed link RS080N_B001_J3_1
- removed link RS080N_B001_J4_1
- removed link RS080N_B001_J5_1
- removed link RS080N_B001_J6_1
- added link flange, mass 0.1
- added link link_1, mass 462.1631225902342; collision mesh filename=meshes/link_1.stl scale=0.001 0.001 0.001; visual mesh filename=meshes/link_1.stl scale=0.001 0.001 0.001
- added link link_2, mass 357.19504838336593; collision mesh filename=meshes/link_2.stl scale=0.001 0.001 0.001; visual mesh filename=meshes/link_2.stl scale=0.001 0.001 0.001
- added link link_3, mass 238.65060564579403; collision mesh filename=meshes/link_3.stl scale=0.001 0.001 0.001; visual mesh filename=meshes/link_3.stl scale=0.001 0.001 0.001
- added link link_4, mass 154.12824627446923; collision mesh filename=meshes/link_4.stl scale=0.001 0.001 0.001; visual mesh filename=meshes/link_4.stl scale=0.001 0.001 0.001
- added link link_5, mass 14.869318086193221; collision mesh filename=meshes/link_5.stl scale=0.001 0.001 0.001; visual mesh filename=meshes/link_5.stl scale=0.001 0.001 0.001
- added link link_6, mass 2.5308375706710504; collision mesh filename=meshes/link_6.stl scale=0.001 0.001 0.001; visual mesh filename=meshes/link_6.stl scale=0.001 0.001 0.001
- added link tool0, mass 0.01
Joints:
- removed joint j1
- removed joint j2
- removed joint j3
- removed joint j4
- removed joint j5
- removed joint j6
- added joint joint_1: type revolute, parent base_link, child link_1, origin xyz=0.0 0.0 0.249 rpy=0 0 0, axis 0.0 0.0 1.0, limit lower=-3.14159 upper=3.14159 effort=1000 velocity=2.181
- added joint joint_2: type revolute, parent link_1, child link_2, origin xyz=0.035 0.15 0.431 rpy=0 0 0, axis 0.0 1.0 0.0, limit lower=-2.268 upper=2.268 effort=1000 velocity=2.181
- added joint joint_3: type revolute, parent link_2, child link_3, origin xyz=0.087 0.0 0.87 rpy=0 0 0, axis 0.0 1.0 0.0, limit lower=-3.92699 upper=1.22173 effort=700 velocity=2.444
- added joint joint_4: type revolute, parent link_3, child link_4, origin xyz=-0.122 0.0 0.27 rpy=0 0 0, axis 1.0 0.0 0.0, limit lower=-3.14159 upper=3.14159 effort=300 velocity=3.491
- added joint joint_5: type revolute, parent link_4, child link_5, origin xyz=-0.0595 0.0 0.81 rpy=0 0 0, axis 0.0 1.0 0.0, limit lower=-2.268 upper=2.268 effort=200 velocity=3.491
- added joint joint_6: type revolute, parent link_5, child link_6, origin xyz=0.0595 0.0 0.1265 rpy=0 0 0, axis 1.0 0.0 0.0, limit lower=-6.28319 upper=6.28319 effort=100 velocity=3.491
- added joint joint_flange: type fixed, parent link_6, child flange, origin xyz=0 0 0 rpy=0 1.57 0
- added joint joint_tool0: type fixed, parent flange, child tool0, origin xyz=0 0 0 rpy=0 0 0
