Commit message: IRB1200H770 tests + fmt

File: library/ABB/IRB1200H_7_70_STD_v1/IRB1200H_7_70_STD.urdf (robot description, URDF)
Before this commit: robot IRB1200H_7_70_STD, 9 links, 8 joints
Joints:
- joint joint_1: origin xyz=0.0 0.0 0.219 rpy=0 0 0 -> xyz=0.0 0.0 0.0 rpy=0 0 0
- joint joint_2: axis 0.0 -1.0 0.0 -> 0.0 1.0 0.0; origin xyz=0.0 -0.0615 0.1801 rpy=0 0 0 -> xyz=0.0 0.0 0.399 rpy=0 0 0
- joint joint_3: axis 0.0 -1.0 0.0 -> 0.0 1.0 0.0; origin xyz=0.0 0.0005 0.35 rpy=0 0 0 -> xyz=0.0 0.0 0.350 rpy=0 0 0
- joint joint_4: axis -1.0 0.0 1.7e-05 -> 1.0 0.0 1.7e-05; origin xyz=0.1655 0.06088 0.041999 rpy=0 0 0 -> xyz=0.0 0.0 0.042 rpy=0 0 0
- joint joint_5: axis 0.0 -1.0 0.0 -> 0.0 1.0 0.0; origin xyz=0.1855 0.025499 1e-06 rpy=0 0 0 -> xyz=0.351 0.0 0.0 rpy=0 0 0
- joint joint_6: origin xyz=0.0855 -0.025383 0.0 rpy=0 0 0 -> xyz=0.82 0.0 0.0 rpy=0 0 0

Commit message: IRB1200H links correct

File: library/ABB/IRB1200H_7_70_STD_v1/IRB1200H_7_70_STD.urdf (robot description, URDF)
Before this commit: robot IRB1200H_7_70_STD, 9 links, 8 joints
Joints:
- joint joint_6: origin xyz=0.82 0.0 0.0 rpy=0 0 0 -> xyz=0.082 0.0 0.0 rpy=0 0 0

Commit message: Kawasaki RS Models (#18)

File: library/ABB/IRB1200H_7_70_STD_v1/IRB1200H_7_70_STD.urdf (robot description, URDF)
Before this commit: robot IRB1200H_7_70_STD, 9 links, 8 joints
Joints:
- joint joint_1: origin xyz=0.0 0.0 0.219 rpy=0 0 0 -> xyz=0.0 0.0 0.0 rpy=0 0 0
- joint joint_2: axis 0.0 -1.0 0.0 -> 0.0 1.0 0.0; origin xyz=0.0 -0.0615 0.1801 rpy=0 0 0 -> xyz=0.0 0.0 0.399 rpy=0 0 0
- joint joint_3: axis 0.0 -1.0 0.0 -> 0.0 1.0 0.0; origin xyz=0.0 0.0005 0.35 rpy=0 0 0 -> xyz=0.0 0.0 0.350 rpy=0 0 0
- joint joint_4: axis -1.0 0.0 1.7e-05 -> 1.0 0.0 1.7e-05; origin xyz=0.1655 0.06088 0.041999 rpy=0 0 0 -> xyz=0.0 0.0 0.042 rpy=0 0 0
- joint joint_5: axis 0.0 -1.0 0.0 -> 0.0 1.0 0.0; origin xyz=0.1855 0.025499 1e-06 rpy=0 0 0 -> xyz=0.351 0.0 0.0 rpy=0 0 0
- joint joint_6: origin xyz=0.0855 -0.025383 0.0 rpy=0 0 0 -> xyz=0.082 0.0 0.0 rpy=0 0 0
