Commit message: 1520 and 1010

File: library/ABB/IRB1010_1_5kg_370_v1/IRB1010_1_5kg_370.urdf (robot description, URDF)
Before this commit: robot IRB1010_1_5kg_370, 7 links, 6 joints
Links:
- removed link link_1_1
- removed link link_2_1
- removed link link_3_1
- removed link link_4_1
- removed link link_5_1
- removed link link_6_1
- added link flange
- added link link_1, mass 9.047546395498204; collision mesh filename=meshes/link_1.stl scale=0.001 0.001 0.001; visual mesh filename=meshes/link_1.stl scale=0.001 0.001 0.001
- added link link_2, mass 14.853907261172468; collision mesh filename=meshes/link_2.stl scale=0.001 0.001 0.001; visual mesh filename=meshes/link_2.stl scale=0.001 0.001 0.001
- added link link_3, mass 8.779035232978092; collision mesh filename=meshes/link_3.stl scale=0.001 0.001 0.001; visual mesh filename=meshes/link_3.stl scale=0.001 0.001 0.001
- added link link_4, mass 5.919741496574066; collision mesh filename=meshes/link_4.stl scale=0.001 0.001 0.001; visual mesh filename=meshes/link_4.stl scale=0.001 0.001 0.001
- added link link_5, mass 3.9451158074034915; collision mesh filename=meshes/link_5.stl scale=0.001 0.001 0.001; visual mesh filename=meshes/link_5.stl scale=0.001 0.001 0.001
- added link link_6, mass 0.18055793093363143; collision mesh filename=meshes/link_6.stl scale=0.001 0.001 0.001; visual mesh filename=meshes/link_6.stl scale=0.001 0.001 0.001
- added link tool0
Joints:
- removed joint j1
- removed joint j2
- removed joint j3
- removed joint j4
- removed joint j5
- removed joint j6
- added joint flange-tool0: type fixed, parent flange, child tool0, origin xyz=0.0 0.0 0.0 rpy=0 0 0
- added joint joint_1: type revolute, parent base_link, child link_1, origin xyz=0.0 0.0 0.123 rpy=0 0 0, axis 0.0 0.0 -1.0, limit lower=-2.9671 upper=2.9671 effort=250 velocity=5.5851
- added joint joint_2: type revolute, parent link_1, child link_2, origin xyz=-0.0587 0.0 0.067 rpy=0 0 0, axis -1.0 0.0 0.0, limit lower=-1.3080 upper=2.1817 effort=200 velocity=5.5851
- added joint joint_3: type revolute, parent link_2, child link_3, origin xyz=0.1195 0.0 0.185 rpy=0 0 0, axis -1.0 0.0 0.0, limit lower=-3.1416 upper=0.8727 effort=150 velocity=6.5449
- added joint joint_4: type revolute, parent link_3, child link_4, origin xyz=-0.0608 0.0553 0.0 rpy=0 0 0, axis 0.0 -1.0 0.0, limit lower=-2.9671 upper=2.9671 effort=100 velocity=8.7266
- added joint joint_5: type revolute, parent link_4, child link_5, origin xyz=-0.0405 0.1297 0.0 rpy=0 0 0, axis -1.0 0.0 0.0, limit lower=-2.1817 upper=2.1817 effort=80 velocity=8.1995
- added joint joint_6: type revolute, parent link_5, child link_6, origin xyz=0.0405 0.0383 0.0 rpy=0 0 0, axis 0.0 -1.0 0.0, limit lower=-6.2832 upper=6.2832 effort=60 velocity=8.7266
- added joint joint_6-flange: type fixed, parent link_6, child flange, origin xyz=0.0 -0.0383 0.0 rpy=0 0 0

File: library/ABB/IRB1520ID_4_150_v1/IRB1520ID_4_150.urdf (robot description, URDF)
Before this commit: robot IRB1520ID_4_150, 7 links, 6 joints
Links:
- removed link link_1_1
- removed link link_2_1
- removed link link_3_1
- removed link link_4_1
- removed link link_5_1
- removed link link_6_1
- added link flange
- added link link_1, mass 140.431105262512; collision mesh filename=meshes/link_1.stl scale=0.001 0.001 0.001; visual mesh filename=meshes/link_1.stl scale=0.001 0.001 0.001
- added link link_2, mass 41.09408994963129; collision mesh filename=meshes/link_2.stl scale=0.001 0.001 0.001; visual mesh filename=meshes/link_2.stl scale=0.001 0.001 0.001
- added link link_3, mass 87.68237861319876; collision mesh filename=meshes/link_3.stl scale=0.001 0.001 0.001; visual mesh filename=meshes/link_3.stl scale=0.001 0.001 0.001
- added link link_4, mass 21.10958519516661; collision mesh filename=meshes/link_4.stl scale=0.001 0.001 0.001; visual mesh filename=meshes/link_4.stl scale=0.001 0.001 0.001
- added link link_5, mass 4.145062543835652; collision mesh filename=meshes/link_5.stl scale=0.001 0.001 0.001; visual mesh filename=meshes/link_5.stl scale=0.001 0.001 0.001
- added link link_6, mass 0.7222246780605773; collision mesh filename=meshes/link_6.stl scale=0.001 0.001 0.001; visual mesh filename=meshes/link_6.stl scale=0.001 0.001 0.001
- added link tool0
Joints:
- removed joint j1
- removed joint j2
- removed joint j3
- removed joint j4
- removed joint j5
- removed joint j6
- added joint flange-tool0: type fixed, parent flange, child tool0, origin xyz=0.0 0.0 0.0 rpy=0 0 0
- added joint joint_1: type revolute, parent base_link, child link_1, origin xyz=0.0 0.0 0.179 rpy=0 0 0, axis -0.0 -0.0 1.0, limit lower=-2.967 upper=2.967 effort=250 velocity=2.2689
- added joint joint_2: type revolute, parent link_1, child link_2, origin xyz=0.16 -0.101 0.274 rpy=0 0 0, axis 0.0 -1.0 -0.0, limit lower=-1.571 upper=2.618 effort=200 velocity=2.4435
- added joint joint_3: type revolute, parent link_2, child link_3, origin xyz=0.0 -0.02 0.59 rpy=0 0 0, axis 0.0 -1.0 -0.0, limit lower=-1.745 upper=1.396 effort=180 velocity=2.4435
- added joint joint_4: type revolute, parent link_3, child link_4, origin xyz=0.217 0.121676 0.2 rpy=0 0 0, axis -1.0 -0.0 0.0, limit lower=-2.705 upper=2.705 effort=100 velocity=5.5851
- added joint joint_5: type revolute, parent link_4, child link_5, origin xyz=0.506 0.051824 0.0 rpy=0 0 0, axis 0.0 -1.0 -0.0, limit lower=-2.356 upper=2.356 effort=80 velocity=6.6323
- added joint joint_6: type revolute, parent link_5, child link_6, origin xyz=0.189629 -0.0525 0.0 rpy=0 0 0, axis 1.0 0.0 0.0, limit lower=-3.491 upper=3.491 effort=50 velocity=8.0285
- added joint joint_6-flange: type fixed, parent link_6, child flange, origin xyz=0.0 0.0 0.0 rpy=0 0 0

Commit message: 1010

File: library/ABB/IRB1010_1_5kg_370_v1/IRB1010_1_5kg_370.urdf (robot description, URDF)
Before this commit: robot IRB1010_1_5kg_370, 9 links, 8 joints
Joints:
- joint joint_1: axis 0.0 0.0 -1.0 -> 0.0 0.0 1.0; origin xyz=0.0 0.0 0.123 rpy=0 0 0 -> xyz=0.0 0.0 0.0 rpy=0 0 0
- joint joint_2: axis -1.0 0.0 0.0 -> 0.0 1.0 0.0; origin xyz=-0.0587 0.0 0.067 rpy=0 0 0 -> xyz=0.0 0.0 0.190 rpy=0 0 0
- joint joint_3: axis -1.0 0.0 0.0 -> 0.0 1.0 0.0; origin xyz=0.1195 0.0 0.185 rpy=0 0 0 -> xyz=0.0 0.0 0.185 rpy=0 0 0
- joint joint_4: axis 0.0 -1.0 0.0 -> 1.0 0.0 0.0; origin xyz=-0.0608 0.0553 0.0 rpy=0 0 0 -> xyz=0.0 0.0 0.0 rpy=0 0 0
- joint joint_5: axis -1.0 0.0 0.0 -> 0.0 1.0 0.0; origin xyz=-0.0405 0.1297 0.0 rpy=0 0 0 -> xyz=0.185 0.0 0.0 rpy=0 0 0
- joint joint_6: axis 0.0 -1.0 0.0 -> 1.0 0.0 0.0; origin xyz=0.0405 0.0383 0.0 rpy=0 0 0 -> xyz=0.045 0.0 0.0 rpy=0 0 0
- joint joint_6-flange: origin xyz=0.0 -0.0383 0.0 rpy=0 0 0 -> xyz=0.0 0.0 0.0 rpy=0 0 0
